File: Rev_1/ECAD/power_board/power_board.kicad_sch (KiCad schematic)
At the start: 16 parts, among them Q1 NMOS, Q2 NMOS

Commit message: Fundemental function down
Parts:
- removed C1, C2, C3: C, symbol Device:C
- removed D3, D4, D5, D6, D7, D8: D, symbol Device:D
- removed Q1, Q2: NMOS, symbol Simulation_SPICE:NMOS
- removed TR1: ADT1-1WT, RF_Mini-Circuits:Mini-Circuits_CD542_H2.84mm, symbol Transformer:ADT1-1WT
- added C1, C17: 680u, Capacitor_THT:CP_Radial_D35.0mm_P10.00mm_SnapIn, symbol Device:C_Polarized
- added C100, C18, C19, C28, C29, C3, C30, C31, C32, C33: 2m2, Capacitor_THT:CP_Radial_D30.0mm_P10.00mm_SnapIn, symbol Device:C_Polarized
- added C15, C?: 1u, symbol Device:C_Small
- added C16: 100n, symbol Device:C_Small
- added C2, C? (x2): 1u, Capacitor_SMD:C_0805_2012Metric, symbol Device:C_Small
- added D16, D17: BYG20J, Diode_SMD:D_SMA, symbol Device:D
- added D3: KBPC3510W, Diode_THT:Diode_Bridge_GeneSiC_KBPC_W, symbol Diode_Bridge:KBPC3510W
- added D4, D5, D6: schottky, Package_TO_SOT_SMD:TO-263-2, symbol Device:D_Schottky_Dual_CommonAnode_AKK_Split
- added J1: Screw_Terminal_01x03, TerminalBlock_Phoenix:TerminalBlock_Phoenix_MKDS-3-3-5.08_1x03_P5.08mm_Horizontal, symbol Connector:Screw_Terminal_01x03
- added Q1, Q2: IPZA60R070CM8XKSA1, Package_TO_SOT_THT:TO-247-4_Vertical, symbol filip:NMOS_DRIVER_SOURCE
- added Q5, Q6: NMOS, symbol Simulation_SPICE:NMOS
- added Q?: NPN, symbol Simulation_SPICE:NPN
- added R11: 0, symbol Device:R
- added R12, R13: 1k, Resistor_SMD:R_0805_2012Metric, symbol Device:R
- added R19: 5, symbol Device:R
- added R20: R_boot, symbol Device:R
- added R21, R22: 3, symbol Device:R
- added R23, R24: 20m, symbol Device:R_Shunt
- added R32, R33: 10k, Resistor_SMD:R_1206_3216Metric, symbol Device:R
- added R6, R? (x2): 4k7, Resistor_SMD:R_0805_2012Metric, symbol Device:R
- added R7, R?: 10k, Resistor_SMD:R_0805_2012Metric, symbol Device:R
- added R?: 100k, symbol Device:R_Small
- added R?: 100k, symbol Device:R
- added R? (x4): 330, symbol Device:R
- added R?: 4k7, symbol Device:R
- added U1: UCC27714D, Package_SO:SOIC-14_3.9x8.7mm_P1.27mm, symbol Driver_FET:UCC27714D
- added U10, U11: PC837, Package_DIP:DIP-12_W7.62mm, symbol Isolator:PC837
- added U11: B66398W1024T1, filip:ETD59, symbol filip:ETD59
- added U14: ETD59, filip:ETD59, symbol filip:ETD59-Center-Tap
- added U2: LMV393, symbol Comparator:LMV393
- added U?: NE555D, Package_SO:SOIC-8_3.9x4.9mm_P1.27mm, symbol Timer:NE555D
- added U?: ISO6720BD, Package_SO:SOIC-8_3.9x4.9mm_P1.27mm, symbol Isolator:ISO6720BD
- L2: renamed from L1; value L -> 220u
- L3: renamed from L2; value L -> 220u
Connections:
- net GND: now also Q?.3 (E), R?.2; no longer D2.2 (A)
- net L_SW_NODE: now reaches D1.2 (A)
- net L_SW_NODE: now also Q1.1 (D), U14.13 (P2)
- net H_SW_NODE: now reaches D2.1 (K)
- net H_SW_NODE: now also Q2.2 (S), U14.1 (P1)
- net VBUS: now reaches D1.1 (K)
- net VBUS: now also C1.1, C17.1, D3.1 (+), Q2.1 (D)
- net at L2.1: now also D4.2 (K), D5.2 (K), D6.2 (K), U14.19, U14.9
- net at L3.1: now also D4.1 (A), D5.1 (A), D6.1 (A), U14.15, U14.5
- net -70V: now reaches L3.2
- net -70V: now also C19.2, C29.2, C3.2, C31.2, C33.2, R33.2
- net +70V: now reaches L2.2
- net +70V: now also C100.1, C18.1, C28.1, C30.1, C32.1, R32.1
- new net: C100.2, C18.2, C19.1, C28.2, C29.1, C3.1, C30.2, C31.1, C32.2, C33.1, R24.1, R32.2, R33.1
- new net: D5.1 (A), D5.3 (K), U14.14 (S2)
- new net: D4.1 (A), D4.3 (K), U14.26 (S1)
- new net: Q1.2 (S), R23.1
- new net: Q?.2 (B), R?.1, R?.2
- new net: C?.1, R?.2, U?.6 (THRES), U?.7 (DISCH)
- new net: R13.2, U10.10
- new net: R?.2, U10.3
- new net: R?.2, U10.1
- new net: C?.1, R?.1, R?.2
- new net: C?.1, R6.1, R?.2
- new net: Q2.4 (G), R21.2
- new net: C15.1, R19.2, R20.1, U1.7 (VDD)
- new net: D16.2 (A), Q5.2 (G), Q6.1 (D), R20.2
- new net: R?.2, U10.5
- new net: C16.2, D16.1 (K), U1.13 (HB)
- new net: D17.1 (K), Q5.1 (D)
- new net: R?.2, U11.1
- new net: Q1.4 (G), R22.2
- new net +12V_Primary: R19.1
- new net +3V3_Secondary: R7.1, R?.1, U?.1 (VCC1)
- new net +5V_Primary: R12.1, R13.1, R?.1, U?.4 (~{RST}), U?.8 (VCC), U?.8 (VCC2)
- new net AC_L: J1.1 (Pin_1)
- new net AC_N: J1.2 (Pin_2)
- new net EN/NC: Q?.1 (C), U1.4 (EN/NC)
- new net Earth_Protective: J1.3 (Pin_3)
- new net GATE_DRIVER_HI: U1.1 (HI), U?.7 (OUTA)
- new net GATE_DRIVER_LI: U1.2 (LI), U?.6 (OUTB)
- new net GND1: C1.2, C17.2, D2.2 (A), D3.3 (-), R11.2, R23.4
- new net GND2: D6.1 (A), D6.3 (K), R24.4, U14.20 (SC)
- new net HS: C16.1, D17.2 (A), Q2.3 (DS), U1.11 (HS)
- new net H_SW: R21.1, U1.12 (HO)
- new net Input Filter And Slow Start/AC_L_OUT: D3.4
- new net Input Filter And Slow Start/AC_N_OUT: D3.2
- new net LO_SW: Q6.2 (G), U1.6 (LO)
- new net LS: Q1.3 (DS), U1.5 (COM)
- new net L_SW: R22.1
- new net PRIM_CURRENT_PWM: R7.2, R?.1, U10.8
- new net PRIM_CURRENT_SENSE: U2.3 (+)
- new net PRIM_CURRENT_VREF: C2.1, R6.2, U2.2 (-)
- new net PRIM_MUX_SELECT: R12.2, U10.12
- new net PRIM_OCP: R?.1, R?.1, U?.3 (OUT)
- new net PRIM_SGND: C15.2, C2.2, C?.2, C?.2, C?.2, Q5.3 (S), Q6.3 (S), R11.1, U1.3 (VSS), U10.11, U10.7, U10.9, U11.2, U?.1 (GND), U?.5 (GND2)
- new net PRIM_SHUNT_H: R23.2
- new net PRIM_SHUNT_L: R23.3
- new net SEC_SGND: U10.2, U10.4, U10.6, U11.11, U?.4 (GND1)
- new net SEC_SHUNT_H: R24.2
- new net SEC_SHUNT_L: R24.3
- new net ~{PRIM_OCP}: R?.2, U11.12
- new net ~{TRIG}: U2.1, U?.2 (TRIG)
- no-connect marks 0 -> 1
Other:
- added sheet Current Sensing (current_sense.kicad_sch)
- added sheet Input Filter And Slow Start (ac_input_filter.kicad_sch)
- added sheet MCU (mcu.kicad_sch)
- added sheet SR Latch (sr_latch.kicad_sch)
- added sheet Startup Power (startup_power.kicad_sch)
- note added: "621-STPF1040CTW - Needs heatsink"
- note added: "C_boot (C16) should be at least 10 times larger than the equivalent gate capacitance (C_g) of your MOSFET"
- note added: "Industrial-Relays-OJS-SS-112HEF_SPST-NO"
- note added: "MOSFET: IPZA60R070CM8XKSA1"
- note added: "OCP"
- note added: "PRIM -> SEC"
- note added: "Pullup resistor will affect rise time"
- note added: "SEC -> PRIM"
- note added: "T = 1.1RC"
- note added: "Trigger Realy in about 100ms from start to prevent burnout. Dont deliver power without relay being connected"
- moved on the sheet: D1, D2, L2, L3

Commit message: Assign footprints
Parts:
- removed C? (x2): 1u, Capacitor_SMD:C_0805_2012Metric, symbol Device:C_Small
- removed R6, R? (x2): 4k7, Resistor_SMD:R_0805_2012Metric, symbol Device:R
- added C1, C10, C15, C16, C25, C7, C84, C9: 100n, Capacitor_SMD:C_0805_2012Metric, symbol Device:C_Small
- added C11, C12: C_Small, symbol Device:C_Small
- added C26, C27, C28: 1u, Capacitor_SMD:C_0805_2012Metric, symbol Device:C_Small
- added D10, D11, D12, D13, D14, D15, D16, D9: LED, symbol Device:LED
- added J2: Conn_01x09_Socket, Connector_PinHeader_1.27mm:PinHeader_1x09_P1.27mm_Horizontal, symbol Connector:Conn_01x09_Socket
- added R110, R111: 0, Resistor_SMD:R_0603_1608Metric, symbol Device:R_Small
- added R112, R113: 10k, Resistor_SMD:R_0805_2012Metric, symbol Device:R_Small
- added R19, R20: R_Small, symbol Device:R_Small
- added R22, R23, R24, R25, R26, R27, R28, R29: 5k1, Resistor_SMD:R_0805_2012Metric, symbol Device:R
- added R32, R33, R34: 4k7, Resistor_SMD:R_0805_2012Metric, symbol Device:R
- added R4: 1k, symbol Device:R_Small
- added RV1: 100k, symbol Device:R_Potentiometer
- added U10, U11: NMUX1308PW, Package_SO:TSSOP-16_4.4x5mm_P0.65mm, symbol Analog_Switch:NMUX1308PW
- added U12: LMV393, symbol Comparator:LMV393
- added unit 3 of U3
- added U8, U9: 74HC595, symbol 74xx:74HC595
- C6: renamed from C16; footprint (none) -> Capacitor_SMD:C_0805_2012Metric
- R18: renamed from R23; value 20m -> 10m
- R21: renamed from R24; value 20m -> 15m
- R30: renamed from R32; value 10k -> LOAD
- R31: renamed from R33; value 10k -> LOAD
- R7: value 10k -> 1k
- gave numbers to parts that had none: 12
- renumbered C100 to C13, C3 to C14, C18 to C17, C19 to C18, C28 to C19, C29 to C20, C30 to C21, C31 to C22, C32 to C23, C33 to C24, C15 to C4, C17 to C5, C1 to C8, D3 to D1, D16 to D2, D17 to D3, D2 to D4, D1 to D5, D4 to D6, D5 to D7, D6 to D8, L2 to L1, L3 to L2, Q5 to Q2, Q6 to Q3, Q2 to Q4, Q1 to Q5, R19 to R13, R20 to R14, R11 to R15, R21 to R16, R22 to R17, R12 to R5, R13 to R6, U10 to U1, U11 to U13, U2 to U3, U11 to U4, U1 to U6, U14 to U7
Connections:
- net GND is gone; now on net PRIM_SGND: Q1.3 (E), R10.2
- net +3V3_Secondary: now also C10.1, C15.1, C16.1, C25.1, C9.1, U10.16 (V_{CC}), U11.16 (V_{CC}), U12.8 (V+), U8.10 (~{SRCLR}), U8.16 (VCC), U9.10 (~{SRCLR}), U9.16 (VCC)
- net +5V_Primary: now also C1.1, C7.1, RV1.1, U3.8 (V+)
- net GATE_DRIVER_HI: now also U2.2 (INA); no longer U2.7 (OUTA)
- net GATE_DRIVER_LI: no longer U2.6 (OUTB)
- net LO_SW: now also R110.1; no longer Q3.2 (G)
- net PRIM_CURRENT_VREF: now also RV1.2
- net PRIM_MUX_SELECT: now also R1.1; no longer R5.2, U1.12
- net PRIM_SGND: now also C1.2, C7.2, C84.2, R112.2, R113.2, R4.2, U3.4 (V-)
- net SEC_SGND: now also C10.2, C15.2, C16.2, C25.2, C26.2, C27.2, C28.2, C9.2, D10.1 (K), D11.1 (K), D12.1 (K), D13.1 (K), D14.1 (K), D15.1 (K), D16.1 (K), D9.1 (K), J2.9 (Pin_9), U10.8 (GND), U11.8 (GND), U12.4 (V-), U8.13 (~{OE}), U8.8 (GND), U9.13 (~{OE}), U9.8 (GND)
- net VBUS: now also D3.1 (K), Q2.1 (D)
- net at D7.1 (A), D7.3 (K), U7.14 (S2): now also C12.1
- net at D6.1 (A), D7.1 (A), D8.1 (A)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: now also R20.2; no longer U7.15, U7.5
- net at D6.2 (K), D7.2 (K), D8.2 (K)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: now also R19.2; no longer U7.19, U7.9
- net at D6.1 (A), D6.3 (K), U7.26 (S1): now also C11.1
- net ~{RELAY_SOFT_SWITCH}: now reaches R6.2, U1.10
- net at C4.1, R13.2, R14.1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: now also C84.1
- net at D2.2 (A), R14.2: now also R111.1; no longer Q2.2 (G), Q3.1 (D)
- net RELAY_SWITCH: now reaches R3.1
- net GATE_DRIVER_LO: now reaches U2.3 (INB)
- net RELAY_SOFT_SWITCH: now reaches R2.1
- net PRIM_CURRENT_PWM renamed ~{RELAY_SWITCH}
- new net: C26.1, R32.2, R33.1
- new net: C27.1, R33.2, R34.1
- new net: Q3.2 (G), R110.2, R112.1
- new net: D14.2 (A), R27.2
- new net: C11.2, R19.1
- new net: R26.1, U9.4 (QE)
- new net: D13.2 (A), R26.2
- new net: R29.1, U9.7 (QH)
- new net: D16.2 (A), R29.2
- new net: R27.1, U9.5 (QF)
- new net: R24.1, U9.2 (QC)
- new net: D11.2 (A), R24.2
- new net: D9.2 (A), R22.2
- new net: D10.2 (A), R23.2
- new net: Q2.2 (G), Q3.1 (D), R111.2, R113.1
- new net: R4.1, RV1.3
- new net: R23.1, U9.1 (QB)
- new net: R22.1, U9.15 (QA)
- new net: R25.1, U9.3 (QD)
- new net: R28.1, U9.6 (QG)
- new net: D15.2 (A), R28.2
- new net: C12.2, R20.1
- new net: D12.2 (A), R25.2
- new net Current Sensing/AD_TEMP_BOARD: U10.13 (Y0)
- new net Current Sensing/AD_TEMP_DIODE1: U10.14 (Y1)
- new net Current Sensing/AD_TEMP_DIODE2: U10.15 (Y2)
- new net Current Sensing/AD_TEMP_DIODE3: U10.12 (Y3)
- new net Current Sensing/AD_TEMP_NMOS_HS: U10.1 (Y4)
- new net Current Sensing/AD_TEMP_NMOS_LS: U10.5 (Y5)
- new net Current Sensing/AD_TEMP_TANSFORMER: U10.2 (Y6)
- new net GATE_DRIVER_HI_ISO: U2.7 (OUTA)
- new net GATE_DRIVER_LO_ISO: U2.6 (OUTB)
- new net QH': U8.9 (QH'), U9.14 (SER)
- new net RCLK: U8.12 (RCLK), U9.12 (RCLK)
- new net S10: U10.11 (S0), U8.15 (QA)
- new net S11: U10.10 (S1), U8.1 (QB)
- new net S12: U10.9 (S2), U8.2 (QC)
- new net S20: U11.11 (S0), U8.4 (QE)
- new net S21: U11.10 (S1), U8.5 (QF)
- new net S22: U11.9 (S2), U8.6 (QG)
- new net SEC_CURRENT_PWM: R32.1
- new net SEC_CURRENT_SENSE: U12.3 (+)
- new net SEC_CURRENT_VREF: C28.1, R34.2, U12.2 (-)
- new net SEC_OCP: U12.1
- new net SER: U8.14 (SER)
- new net SRCLK: U8.11 (SRCLK), U9.11 (SRCLK)
- new net TEMP_MUX1: U10.3 (Z)
- new net TEMP_MUX2: U11.3 (Z)
- new net Y0: J2.1 (Pin_1), U11.13 (Y0)
- new net Y1: J2.2 (Pin_2), U11.14 (Y1)
- new net Y2: J2.3 (Pin_3), U11.15 (Y2)
- new net Y3: J2.4 (Pin_4), U11.12 (Y3)
- new net Y4: J2.5 (Pin_5), U11.1 (Y4)
- new net Y5: J2.6 (Pin_6), U11.5 (Y5)
- new net Y6: J2.7 (Pin_7), U11.2 (Y6)
- new net Y7: J2.8 (Pin_8), U11.4 (Y7)
- new net ~{E}1: U10.6 (~{E}), U8.3 (QD)
- new net ~{E}2: U11.6 (~{E}), U8.7 (QH)
- new net ~{PRIM_MUX_SELECT}: R5.2, U1.12
- no-connect marks 1 -> 3
Other:
- sheet Current Sensing ports: added AD_TEMP_BOARD, AD_TEMP_DIODE1, AD_TEMP_DIODE2, AD_TEMP_DIODE3, AD_TEMP_NMOS_HS, AD_TEMP_NMOS_LS, AD_TEMP_TANSFORMER, MUX_OUT, SEC_NEG_VOLTAGE, SEC_POS_VOLTAGE; removed none
- sheet Input Filter And Slow Start ports: added RELAY_SOFT_SWITCH; removed none
- sheet MCU ports: added PB0, PB1, PB2, RCLK, SER, SRCLK, TIM1_BKN, TIM1_CH1, TIM1_CH2, TIM2_CH2; removed none
- note added: "* Output diodes should be soft recovery diodes * RC snubber on the output diodes to avoid ringing * D1 & D2 Ultrafast recovery diodes rated >600V and can handle the peak magnetizing current."
- note added: "*MCU heartbeat *Soft start *Power stage enabled *Output rails OK *Current limit active *Thermal Warning *Protection trip"
- note added: "5k1 Ohms"
- note added: "Gate Driver"
- note added: "Green LEDs"
- note added: "OCP Primary"
- note added: "OCP Secondary"
- note removed: "* Output diodes should be soft recovery diodes * RC snubber on the output diodes to avoid ringing"
- moved on the sheet: C13, C14, C17, C18, C19, C2, C20, C21, C22, C23, C24, C3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
