File: Rev_1/ECAD/power_board/current_sense.kicad_sch (KiCad schematic)
At the start: 78 parts, among them U3 INA180A4

Commit message: Assign footprints
Parts:
- removed U3, U?: INA180A4, Package_TO_SOT_SMD:SOT-23-5, symbol Amplifier_Current:INA180A4
- added C41, C42, C44: 100n, Capacitor_SMD:C_0805_2012Metric, symbol Device:C_Small
- added D19, D24, D26: BAT54S, Package_TO_SOT_SMD:SOT-23, symbol Diode:BAT54S
- added R55: 3k3, symbol Device:R_Small
- added R56, R57, R58: 27k, symbol Device:R_Small
- added R61, R66, R68: 3k3, symbol Device:R
- added R70: 1k, symbol Device:R
- added U14: INA180A2, Package_TO_SOT_SMD:SOT-23-5, symbol Amplifier_Current:INA180A2
- added U15: INA180A1, Package_TO_SOT_SMD:SOT-23-5, symbol Amplifier_Current:INA180A1
- added U18: LM358, symbol Amplifier_Operational:LM358
- C31: renamed from C34; now not fitted
- C33: renamed from C35; now not fitted
- C47, C48: renamed from C?; value 120p -> 100n; footprint (none) -> Capacitor_SMD:C_0805_2012Metric
- gave numbers to parts that had none: 66
- renumbered C11 to C35, R25 to R37, R26 to R38, R27 to R45, R28 to R46, R31 to R47
Connections:
- net PRIMARY_BUS_VOLTAGE is gone; now on net PRIM_BUS_VOLTAGE: D28.3 (COM), R81.2
- net +: now also U14.3 (+), U15.3 (+)
- net +3V3: now also D26.2 (K)
- net +3V3_Secondary: now also C36.1, C42.1, D19.2 (K), U15.5 (V+), U18.8 (V+)
- net +5V_Secondary: now also C35.1, U14.5 (V+)
- net -: now also U14.4 (-), U15.4 (-)
- net AD_TEMP_DIODE3: no longer D25.3 (COM), R65.2
- net PRIMARY_CURRENT_SENSE: now also U14.1, U15.1
- net PRIM_SGND: now also U14.2 (GND), U15.2 (GND)
- net SEC_CURRENT_SENSE: now also D19.3 (COM)
- net SEC_SGND: now also C41.2, C42.2, C44.2, D19.1 (A), D24.2 (K), D26.1 (A), R55.2, U18.5 (+)
- removed net +5V: C35.1, C36.1
- new net: R66.2, R68.1, U18.6 (-)
- new net: R68.2, R70.1, U18.7
- new net: C41.1, R55.1, R56.2, R61.1
- new net: D24.3 (COM), R61.2, U18.3 (+)
- new net: R56.1, R57.2
- new net: R57.1, R58.2
- new net: R66.1, U18.1, U18.2 (-)
- new net -5V: C44.1, D24.1 (A), U18.4 (V-)
- new net -70V: R58.1
- new net AD_TEMP_TANSFORMER: D25.3 (COM), R65.2
- new net SEC_NEG_VOLTAGE: D26.3 (COM), R70.2
Other:
- note added: "Gain = 13.34 2.67v@20A"
- note added: "Gain = 33.34 2.57v@8A"
- note added: "Secondary Neg Voltage"
- note added: "Secondary Pos Voltage"
- note removed: "Gain = 50 3.3v@9.5A"
- note removed: "Secondary Voltage"

Commit message: Before PR
Parts:
- added C36, C41: 1u, 16VDC, Capacitor_SMD:C_0805_2012Metric, symbol Device:C_Small
- added D27, D30: BAT54S, Package_TO_SOT_SMD:SOT-23, symbol Diode:BAT54S
- added R66, R77: 3k3, Resistor_SMD:R_0603_1608Metric, symbol Device:R
- added R70, R78: 3k3, Resistor_SMD:R_0603_1608Metric, symbol Device:R_Small
- added TH7, TH9: 10k, Connector_PinHeader_2.54mm:PinHeader_1x02_P2.54mm_Vertical, symbol Device:Thermistor_NTC
- added TP16: PRIM_SHUNT_H, Connector_Pin:Pin_D0.7mm_L6.5mm_W1.8mm_FlatFork, symbol Connector:TestPoint
- added TP17: PRIM_SHUNT_L, Connector_Pin:Pin_D0.7mm_L6.5mm_W1.8mm_FlatFork, symbol Connector:TestPoint
- C22: renamed from C29; value 1u -> 1u, 16VDC; footprint (none) -> Capacitor_SMD:C_0805_2012Metric; Part-DB ID (none) -> 36; Part-DB NAME (none) -> 0805B105K160CT
- C23: renamed from C30; value 1u -> 1u, 16VDC; footprint (none) -> Capacitor_SMD:C_0805_2012Metric; Part-DB ID (none) -> 36; Part-DB NAME (none) -> 0805B105K160CT
- C24: renamed from C31; footprint (none) -> Capacitor_SMD:C_0603_1608Metric
- C25: renamed from C32; footprint (none) -> Capacitor_SMD:C_0603_1608Metric; now not fitted
- C26: renamed from C33; footprint (none) -> Capacitor_SMD:C_0603_1608Metric
- C27: renamed from C34; footprint (none) -> Capacitor_SMD:C_0603_1608Metric
- C28: renamed from C35; value 100n -> 100n, 16VDC; Part-DB ID (none) -> 9; Part-DB NAME (none) -> 0805B104K160CT
- C29: renamed from C36; value 100n -> 100n, 16VDC; Part-DB ID (none) -> 9; Part-DB NAME (none) -> 0805B104K160CT
- C30: renamed from C37; value 1u -> 1u, 16VDC; footprint (none) -> Capacitor_SMD:C_0805_2012Metric; Part-DB ID (none) -> 36; Part-DB NAME (none) -> 0805B105K160CT
- C31: renamed from C38; value 1u -> 1u, 16VDC; footprint (none) -> Capacitor_SMD:C_0805_2012Metric; Part-DB ID (none) -> 36; Part-DB NAME (none) -> 0805B105K160CT
- C32: renamed from C39; value 1u -> 1u, 16VDC; footprint (none) -> Capacitor_SMD:C_0805_2012Metric; Part-DB ID (none) -> 36; Part-DB NAME (none) -> 0805B105K160CT
- C33: renamed from C40; value 1u -> 1u, 16VDC; footprint (none) -> Capacitor_SMD:C_0805_2012Metric; Part-DB ID (none) -> 36; Part-DB NAME (none) -> 0805B105K160CT
- C34: renamed from C41; value 100n -> 100n, 16VDC; Part-DB ID (none) -> 9; Part-DB NAME (none) -> 0805B104K160CT
- C35: renamed from C42; value 100n -> 100n, 16VDC; Part-DB ID (none) -> 9; Part-DB NAME (none) -> 0805B104K160CT
- C37: renamed from C43; value 1u -> 1u, 16VDC; footprint (none) -> Capacitor_SMD:C_0805_2012Metric; Part-DB ID (none) -> 36; Part-DB NAME (none) -> 0805B105K160CT
- C38: renamed from C44; value 100n -> 100n, 16VDC; Part-DB ID (none) -> 9; Part-DB NAME (none) -> 0805B104K160CT
- C39: renamed from C45; footprint (none) -> Capacitor_SMD:C_0603_1608Metric
- C40: renamed from C46; footprint (none) -> Capacitor_SMD:C_0603_1608Metric
- C42: renamed from C47; value 100n -> 100n, 16VDC; Part-DB ID (none) -> 9; Part-DB NAME (none) -> 0805B104K160CT
- C43: renamed from C48; value 100n -> 100n, 16VDC; Part-DB ID (none) -> 9; Part-DB NAME (none) -> 0805B104K160CT
- D19: renamed from D17; Mouser No: (none) -> 637-BAT54S; Part-DB ID (none) -> 92; Part-DB NAME (none) -> BAT54s
- D20: renamed from D18; Mouser No: (none) -> 637-BAT54S; Part-DB ID (none) -> 92; Part-DB NAME (none) -> BAT54s
- D21: renamed from D19; Mouser No: (none) -> 637-BAT54S; Part-DB ID (none) -> 92; Part-DB NAME (none) -> BAT54s
- D22: renamed from D20; Mouser No: (none) -> 637-BAT54S; Part-DB ID (none) -> 92; Part-DB NAME (none) -> BAT54s
- D23: renamed from D21; Mouser No: (none) -> 637-BAT54S; Part-DB ID (none) -> 92; Part-DB NAME (none) -> BAT54s
- D24: renamed from D22; Mouser No: (none) -> 637-BAT54S; Part-DB ID (none) -> 92; Part-DB NAME (none) -> BAT54s
- D25: renamed from D23; Mouser No: (none) -> 637-BAT54S; Part-DB ID (none) -> 92; Part-DB NAME (none) -> BAT54s
- D26: renamed from D24; Mouser No: (none) -> 637-BAT54S; Part-DB ID (none) -> 92; Part-DB NAME (none) -> BAT54s
- D28: renamed from D25; Mouser No: (none) -> 637-BAT54S; Part-DB ID (none) -> 92; Part-DB NAME (none) -> BAT54s
- D29: renamed from D26; Mouser No: (none) -> 637-BAT54S; Part-DB ID (none) -> 92; Part-DB NAME (none) -> BAT54s
- D31: renamed from D27; Mouser No: (none) -> 637-BAT54S; Part-DB ID (none) -> 92; Part-DB NAME (none) -> BAT54s
- D32: renamed from D28; Mouser No: (none) -> 637-BAT54S; Part-DB ID (none) -> 92; Part-DB NAME (none) -> BAT54s
- R39: renamed from R35; footprint (none) -> Resistor_SMD:R_0603_1608Metric; Part-DB ID (none) -> 72; Part-DB NAME (none) -> RK73B1JTTDD332J
- R40: renamed from R36; footprint (none) -> Resistor_SMD:R_0603_1608Metric; Part-DB ID (none) -> 72; Part-DB NAME (none) -> RK73B1JTTDD332J
- R41: renamed from R39; footprint (none) -> Resistor_SMD:R_0805_2012Metric; Part-DB ID (none) -> 28; Part-DB NAME (none) -> WR08X1000FTL
- R42: renamed from R40; footprint (none) -> Resistor_SMD:R_0805_2012Metric; Part-DB ID (none) -> 28; Part-DB NAME (none) -> WR08X1000FTL
- R43: renamed from R37; footprint (none) -> Resistor_SMD:R_0805_2012Metric; Part-DB ID (none) -> 28; Part-DB NAME (none) -> WR08X1000FTL
- R44: renamed from R38; footprint (none) -> Resistor_SMD:R_0805_2012Metric; Part-DB ID (none) -> 28; Part-DB NAME (none) -> WR08X1000FTL
- R45: renamed from R41; footprint (none) -> Resistor_SMD:R_0603_1608Metric; Part-DB ID (none) -> 72; Part-DB NAME (none) -> RK73B1JTTDD332J
- R46: renamed from R42; footprint (none) -> Resistor_SMD:R_0603_1608Metric; Part-DB ID (none) -> 72; Part-DB NAME (none) -> RK73B1JTTDD332J
- R47: renamed from R43; footprint (none) -> Resistor_SMD:R_0603_1608Metric; Part-DB ID (none) -> 72; Part-DB NAME (none) -> RK73B1JTTDD332J
- R48: renamed from R44; footprint (none) -> Resistor_SMD:R_0603_1608Metric; Part-DB ID (none) -> 72; Part-DB NAME (none) -> RK73B1JTTDD332J
- R49: renamed from R45; footprint (none) -> Resistor_SMD:R_0805_2012Metric; Part-DB ID (none) -> 66; Part-DB NAME (none) -> 40819310
- R50: renamed from R46; footprint (none) -> Resistor_SMD:R_0805_2012Metric; Part-DB ID (none) -> 66; Part-DB NAME (none) -> 40819310
- R51: renamed from R47; footprint (none) -> Resistor_SMD:R_0805_2012Metric; Part-DB ID (none) -> 66; Part-DB NAME (none) -> 40819310
- R52: renamed from R48; footprint (none) -> Resistor_SMD:R_0805_2012Metric; Part-DB ID (none) -> 66; Part-DB NAME (none) -> 40819310
- R53: renamed from R49; footprint (none) -> Resistor_SMD:R_0805_2012Metric; Part-DB ID (none) -> 66; Part-DB NAME (none) -> 40819310
- R54: renamed from R50; footprint (none) -> Resistor_SMD:R_0805_2012Metric; Part-DB ID (none) -> 66; Part-DB NAME (none) -> 40819310
- R55: renamed from R51; footprint (none) -> Resistor_SMD:R_0603_1608Metric; Part-DB ID (none) -> 72; Part-DB NAME (none) -> RK73B1JTTDD332J
- R56: renamed from R52; footprint (none) -> Resistor_SMD:R_0603_1608Metric; Part-DB ID (none) -> 72; Part-DB NAME (none) -> RK73B1JTTDD332J
- R57: renamed from R53; footprint (none) -> Resistor_SMD:R_0603_1608Metric; Part-DB ID (none) -> 72; Part-DB NAME (none) -> RK73B1JTTDD332J
- R58: renamed from R54; footprint (none) -> Resistor_SMD:R_0603_1608Metric; Part-DB ID (none) -> 72; Part-DB NAME (none) -> RK73B1JTTDD332J
- R59: renamed from R55; footprint (none) -> Resistor_SMD:R_0603_1608Metric; Part-DB ID (none) -> 72; Part-DB NAME (none) -> RK73B1JTTDD332J
- R60: renamed from R56; footprint (none) -> Resistor_SMD:R_0805_2012Metric
- R61: renamed from R57; footprint (none) -> Resistor_SMD:R_0805_2012Metric
- R62: renamed from R58; footprint (none) -> Resistor_SMD:R_0805_2012Metric
- R63: renamed from R59; footprint (none) -> Resistor_SMD:R_0603_1608Metric; Part-DB ID (none) -> 72; Part-DB NAME (none) -> RK73B1JTTDD332J
- R64: renamed from R60; footprint (none) -> Resistor_SMD:R_0603_1608Metric; Part-DB ID (none) -> 72; Part-DB NAME (none) -> RK73B1JTTDD332J
- R65: renamed from R61; footprint (none) -> Resistor_SMD:R_0603_1608Metric; Part-DB ID (none) -> 72; Part-DB NAME (none) -> RK73B1JTTDD332J
- R67: renamed from R62; footprint (none) -> Resistor_SMD:R_0603_1608Metric; Part-DB ID (none) -> 72; Part-DB NAME (none) -> RK73B1JTTDD332J
- R68: renamed from R63; footprint (none) -> Resistor_SMD:R_0805_2012Metric; Part-DB ID (none) -> 67; Part-DB NAME (none) -> 40819410
- R69: renamed from R64; footprint (none) -> Resistor_SMD:R_0805_2012Metric; Part-DB ID (none) -> 67; Part-DB NAME (none) -> 40819410
- R71: renamed from R65; footprint (none) -> Resistor_SMD:R_0603_1608Metric; Part-DB ID (none) -> 72; Part-DB NAME (none) -> RK73B1JTTDD332J
- R72: renamed from R66; footprint (none) -> Resistor_SMD:R_0603_1608Metric; Part-DB ID (none) -> 72; Part-DB NAME (none) -> RK73B1JTTDD332J
- R73: renamed from R67; footprint (none) -> Resistor_SMD:R_0603_1608Metric
- R74: renamed from R68; footprint (none) -> Resistor_SMD:R_0603_1608Metric; Part-DB ID (none) -> 72; Part-DB NAME (none) -> RK73B1JTTDD332J
- R75: renamed from R69; footprint (none) -> Resistor_SMD:R_0603_1608Metric
- R76: renamed from R70; footprint (none) -> Resistor_SMD:R_0805_2012Metric; Part-DB ID (none) -> 66; Part-DB NAME (none) -> 40819310
- R79: renamed from R71; footprint (none) -> Resistor_SMD:R_0805_2012Metric; Part-DB ID (none) -> 45; Part-DB NAME (none) -> RC0805FR-1068KL
- R80: renamed from R72; footprint (none) -> Resistor_SMD:R_0805_2012Metric; Part-DB ID (none) -> 45; Part-DB NAME (none) -> RC0805FR-1068KL
- R81: renamed from R73; footprint (none) -> Resistor_SMD:R_0805_2012Metric; Part-DB ID (none) -> 45; Part-DB NAME (none) -> RC0805FR-1068KL
- R82: renamed from R74; footprint (none) -> Resistor_SMD:R_0805_2012Metric; Part-DB ID (none) -> 45; Part-DB NAME (none) -> RC0805FR-1068KL
- R83: renamed from R75; footprint (none) -> Resistor_SMD:R_0805_2012Metric; Part-DB ID (none) -> 45; Part-DB NAME (none) -> RC0805FR-1068KL
- R84: renamed from R76; footprint (none) -> Resistor_SMD:R_0603_1608Metric
- R85: renamed from R77; footprint (none) -> Resistor_SMD:R_0805_2012Metric
- R86: renamed from R78; footprint (none) -> Resistor_SMD:R_0805_2012Metric
- R87: renamed from R79; footprint (none) -> Resistor_SMD:R_0805_2012Metric
- R88: renamed from R80; footprint (none) -> Resistor_SMD:R_0603_1608Metric; Part-DB ID (none) -> 72; Part-DB NAME (none) -> RK73B1JTTDD332J
- R89: renamed from R81; footprint (none) -> Resistor_SMD:R_0603_1608Metric; Part-DB ID (none) -> 72; Part-DB NAME (none) -> RK73B1JTTDD332J
- R90: renamed from R82; footprint (none) -> Resistor_SMD:R_0603_1608Metric; Part-DB ID (none) -> 72; Part-DB NAME (none) -> RK73B1JTTDD332J
- TH1, TH2, TH3, TH4, TH5: footprint (none) -> Connector_PinHeader_2.54mm:PinHeader_1x02_P2.54mm_Vertical
- TH8: renamed from TH7; footprint (none) -> Connector_PinHeader_2.54mm:PinHeader_1x02_P2.54mm_Vertical
- U10: renamed from U14; Mouser No: (none) -> INA180A2IDBVR
- U11: renamed from U15; Mouser No: (none) -> INA180A1IDBVR
- U13: renamed from U17; Mouser No: (none) -> 595-AMC1350DWVR
- U14: renamed from U18; footprint (none) -> Package_SO:TSSOP-8_3x3mm_P0.65mm; Mouser No: (none) -> 595-LM358BIPWR
- renumbered U16 to U12, U19 to U15
Connections:
- net +: no longer C24.1, R43.2, U10.3 (+)
- net +3V3_Secondary: now also D29.2 (K), D31.2 (K), D27.2 (K), D30.2 (K), R66.1, R77.1
- net +5V_Primary: now also C28.1, D32.2 (K), U10.5 (V+)
- net +5V_Secondary: no longer C28.1, U10.5 (V+)
- net -: no longer C26.1, R44.2, U10.4 (-)
- net PRIMARY_CURRENT_SENSE: no longer R52.1, U11.1
- net PRIM_SGND: now also D32.1 (A); no longer C25.2, C27.2, C29.2, R54.2, U11.2 (GND)
- net PRIM_SHUNT_H: now also R43.1, TP16.1; no longer R44.1
- net PRIM_SHUNT_L: now also R44.1, TP17.1; no longer R43.1
- net SEC_SGND: now also C25.2, C27.2, C29.2, R54.2, U11.2 (GND), C36.2, C41.2, D27.1 (A), D30.1 (A), TH7.2, TH9.2; no longer D32.1 (A)
- net SEC_SHUNT_H: now also R41.1; no longer R42.1
- net SEC_SHUNT_L: now also R42.1; no longer R41.1
- removed net +3V3: D29.2 (K), D31.2 (K), D32.2 (K)
- new net: C26.1, R44.2, U10.4 (-)
- new net: C36.1, R66.2, R70.1, TH7.1
- new net: C41.1, R77.2, R78.1, TH9.1
- new net: C24.1, R43.2, U10.3 (+)
- new net AD_TEMP_DIODE_PRIM1: D27.3 (COM), R70.2
- new net AD_TEMP_DIODE_PRIM2: D30.3 (COM), R78.2
- new net SECONDARY_CURRENT_SENSE: R52.1, U11.1
Other:
- added sheet HW Protection (hw_protection.kicad_sch)
- note added: "Change to 330p?"
- note added: "Diode PRIM 1"
- note added: "Diode PRIM 2"
- note added: "Look Thorugh This!"
- moved on the sheet: C23, C31, D20, D23, R40, R43, R44, R46, R48, R56, TH2, TH4
