File: Rev_1/ECAD/power_board/mcu.kicad_sch (KiCad schematic)
At the start: 51 parts, among them J2 Conn_ARM_JTAG_SWD_10, J3 USB_C_Receptacle_USB2.0_16P, J4 Conn_01x04_Pin, SW1 SW_Push, SW2 SW_Push, U12 STM32F103C8Tx, U15 USBLC6-2SC6, U16 74HC595

Commit message: Assign footprints
Parts:
- removed C44: 100n, Capacitor_SMD:C_0805_2012Metric, symbol Device:C_Small
- removed D18, D19, D20, D21, D22, D23, D24, D25: LED, symbol Device:LED
- removed R39, R40, R41, R42, R43, R44, R45, R46: 5k1, Resistor_SMD:R_0805_2012Metric, symbol Device:R
- removed U16: 74HC595, symbol 74xx:74HC595
- added C77, C78: 27p, Capacitor_SMD:C_0603_1608Metric, symbol Device:C_Small
- added C82: 100n, Capacitor_SMD:C_0805_2012Metric, symbol Device:C_Small
- added U28: TPS3823-xxDBV, Package_TO_SOT_SMD:SOT-23-5, symbol Power_Supervisor:TPS3823-xxDBV
- added Y1: 8MHz, symbol Device:Crystal_GND3_Small
- C80: renamed from C42; footprint (none) -> Capacitor_SMD:C_0805_2012Metric
- C81: renamed from C43; footprint (none) -> Capacitor_SMD:C_0805_2012Metric
- gave numbers to parts that had none: 8
- renumbered C20 to C72, C36 to C73, C37 to C74, C38 to C75, C39 to C76, C40 to C79, D9 to D38, J2 to J5, R9 to R100, R34 to R101, R35 to R102, R36 to R103, R37 to R104, R38 to R105, R8 to R99, U15 to U26, U12 to U27
Connections:
- net +3V3_Secondary: now also C82.1, U28.5 (V_{DD})
- net RCLK: now also U27.42 (PB6); no longer U27.41 (PB5)
- net SEC_SGND: now also C79.1, C77.1, C78.2, C82.2, U28.2 (GND), Y1.3; no longer C79.2
- net TACHO_1: now also U27.40 (PB4); no longer U27.42 (PB6)
- net TACHO_2: now also U27.41 (PB5); no longer U27.43 (PB7)
- net ~{RST}: now also C79.2, U28.1 (~{RESET}); no longer C79.1, SW1.2
- net PB0: now reaches U27.18 (PB0)
- net PB1: now reaches U27.19 (PB1)
- net PB2: now reaches U27.20 (PB2)
- net WDI: now reaches U27.31 (PA10)
- net WDI: now also U28.4 (WDI)
- net TIM2_CH2: now reaches U27.39 (PB3)
- net RCC_OSC_IN: now reaches U27.5 (PD0)
- net RCC_OSC_IN: now also C77.2, Y1.1
- net RCC_OSC_OUT: now reaches U27.6 (PD1)
- net RCC_OSC_OUT: now also C78.1, Y1.2
- new net ~{MR}: SW1.2, U28.3 (~{MR})
- no-connect marks 7 -> 6
Other:
- note added: "Fans"
- note added: "SWD"
- note added: "Watchdog"
- note removed: "*MCU heartbeat *Soft start *Power stage enabled *Output rails OK *Current limit active *Thermal Warning *Protection trip"
- note removed: "5k1 Ohms"
- note removed: "Green LEDs"
- moved on the sheet: C72, C73, C74, C75, C76, C79, C80, C81, D38, F2, FB1, J3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

Commit message: Before PR
Parts:
- removed J4: Conn_01x04_Pin, Connector_JST:JST_EH_S4B-EH_1x04_P2.50mm_Horizontal, symbol Connector:Conn_01x04_Pin
- added D43, D44, D45: 1N4148, Diode_THT:D_DO-35_SOD27_P7.62mm_Horizontal, symbol Diode:1N4148
- C68: renamed from C72; value 100n -> 100n, 16VDC; Part-DB ID (none) -> 9; Part-DB NAME (none) -> 0805B104K160CT
- C69: renamed from C73; value 100n -> 100n, 16VDC; Part-DB ID (none) -> 9; Part-DB NAME (none) -> 0805B104K160CT
- C70: renamed from C74; value 100n -> 100n, 16VDC; Part-DB ID (none) -> 9; Part-DB NAME (none) -> 0805B104K160CT
- C71: renamed from C75; value 100n -> 100n, 16VDC; Part-DB ID (none) -> 9; Part-DB NAME (none) -> 0805B104K160CT
- C75: renamed from C79; value 100n -> 100n, 16VDC; Part-DB ID (none) -> 9; Part-DB NAME (none) -> 0805B104K160CT
- C76: renamed from C80; value 100n -> 100n, 16VDC; Part-DB ID (none) -> 9; Part-DB NAME (none) -> 0805B104K160CT
- C77: renamed from C81; value 100n -> 100n, 16VDC; Part-DB ID (none) -> 9; Part-DB NAME (none) -> 0805B104K160CT
- C78: renamed from C82; value 100n -> 100n, 16VDC; Part-DB ID (none) -> 9; Part-DB NAME (none) -> 0805B104K160CT
- D42: renamed from D38; footprint (none) -> Diode_SMD:D_SOD-523; Mouser No: (none) -> 637-ESD5B5V0WT; now not fitted
- F2: footprint (none) -> Varistor:RV_Disc_D15.5mm_W5mm_P7.5mm; Mouser No: (none) -> 576-60R050XU
- FB1: footprint (none) -> Inductor_SMD:L_0805_2012Metric
- J3: footprint (none) -> Connector_USB:USB_C_Receptacle_GCT_USB4105-xx-A_16P_TopMnt_Horizontal; Part-DB ID (none) -> 82; Part-DB NAME (none) -> DX07S016JA2R1500
- M1, M2: footprint Connector_JST:JST_PH_B4B-PH-K_1x04_P2.00mm_Vertical -> Connector:FanPinHeader_1x04_P2.54mm_Vertical
- R108: renamed from R100; Part-DB ID (none) -> 67; Part-DB NAME (none) -> 40819410
- R109: renamed from R101; Part-DB ID (none) -> 17; Part-DB NAME (none) -> RT0805DRD075K1L
- R110: renamed from R102; Part-DB ID (none) -> 17; Part-DB NAME (none) -> RT0805DRD075K1L
- R111: renamed from R103; footprint (none) -> Resistor_SMD:R_0603_1608Metric
- R112: renamed from R104; footprint (none) -> Resistor_SMD:R_0603_1608Metric
- R113: renamed from R105; footprint (none) -> Resistor_SMD:R_0603_1608Metric
- R114: renamed from R106; Part-DB ID (none) -> 67; Part-DB NAME (none) -> 40819410
- R115: renamed from R107; Part-DB ID (none) -> 67; Part-DB NAME (none) -> 40819410
- R116: renamed from R108; Part-DB ID (none) -> 67; Part-DB NAME (none) -> 40819410
- R117: renamed from R109; Part-DB ID (none) -> 67; Part-DB NAME (none) -> 40819410
- U23: renamed from U27; Part-DB ID (none) -> 29; Part-DB NAME (none) -> STM32F103C8T6
- U24: renamed from U28; Mouser No: (none) -> 595-TPS3823-25DBVR
- Y1: footprint (none) -> filip:HC-49US
- renumbered C76 to C72, C77 to C73, C78 to C74, J5 to J4, R99 to R107, U26 to U22
Connections:
- net FAN_PWM_1: no longer Q9.1 (G), R115.1
- net FAN_PWM_2: now also Q9.1 (G), R115.1
- net TACHO_1: no longer M2.3 (Tacho)
- net TACHO_2: now also M2.3 (Tacho)
- net TIM1_BKN: now also D43.1 (K), D44.1 (K), D45.1 (K)
- net PWM_1: now reaches M1.4 (PWM), Q8.3 (D), R116.2
- net PC13: now reaches U23.2 (PC13)
- net PA15: now reaches U23.38 (PA15)
- net PWM_2: now reaches M2.4 (PWM), Q9.3 (D), R117.2
- net ADC7 renamed PA7
- net MISO renamed PB14
- net MOSI renamed PB15
- net SCK renamed PB13
- net ~{SS} renamed PB12
- new net TIM1_BKN_0: D43.2 (A)
- new net TIM1_BKN_1: D44.2 (A)
- new net TIM1_BKN_2: D45.2 (A)
- no-connect marks 6 -> 8
