File: Rev_1/ECAD/power_board/power_board.kicad_pcb (KiCad board)
At the start: 2 copper layers, 96 parts, among them J1 Screw_Terminal_01x03, J2 Conn_ARM_JTAG_SWD_10, J4 Conn_01x04_Pin, K1 SPST-NO, Q1 IPZA60R070CM8XKSA1, Q2 IPZA60R070CM8XKSA1, SW1 SW_Push, SW2 SW_Push, T1 063932, U1 UCC27714D, U10 PC837, U11 B66398W1024T1, U12 STM32F103C8Tx, U15 USBLC6-2SC6, U3 INA180A4, U4 PC837, U5 TNY274P, U6 PC817, U7 5V LDO, U8 LMR51430, U9 3v3 LDO

Commit message: Before PR
Parts:
- removed C100: 2m2, Capacitor_THT:CP_Radial_D30.0mm_P10.00mm_SnapIn
- removed the R7 at (154.2, 140.8)
- removed the R7 at (87.9, 116.1)
- removed the R8 at (130.3, 166.4)
- removed the R8 at (87.9, 119.1)
- removed the R9 at (130.3, 169.4)
- removed the R9 at (87.9, 122.0)
- removed TR1: ADT1-1WT, RF_Mini-Circuits:Mini-Circuits_CD542_H2.84mm
- added C10: 100n, Capacitor_SMD:C_0805_2012Metric, F.Cu at (-226.9, -88.7)
- added C13: 2m2, Capacitor_THT:CP_Radial_D30.0mm_P10.00mm_SnapIn, F.Cu at (-390.4, -144.8)
- added C14: 2m2, Capacitor_THT:CP_Radial_D30.0mm_P10.00mm_SnapIn, F.Cu at (-390.4, -113.2)
- added C15: 2m2, Capacitor_THT:CP_Radial_D30.0mm_P10.00mm_SnapIn, F.Cu at (-390.4, -81.7)
- added C16: 2m2, Capacitor_THT:CP_Radial_D30.0mm_P10.00mm_SnapIn, F.Cu at (-390.4, -50.1)
- added C21: 2m2, Capacitor_THT:CP_Radial_D30.0mm_P10.00mm_SnapIn, F.Cu at (-357.9, -50.1)
- added C25: TBD, Capacitor_SMD:C_0603_1608Metric, F.Cu at (-239.3, -73.5)
- added C34: 100n, Capacitor_SMD:C_0805_2012Metric, F.Cu at (-244.9, -53.5)
- added C35: 100n, Capacitor_SMD:C_0805_2012Metric, F.Cu at (-244.9, -50.5)
- added C4: 100n, Capacitor_SMD:C_0805_2012Metric, F.Cu at (133.2, 50.4)
- added C41: 1u, Capacitor_SMD:C_0805_2012Metric, F.Cu at (-240.5, -50.5)
- added C42: 100n, Capacitor_SMD:C_0805_2012Metric, F.Cu at (-240.5, -47.5)
- added C43: 100n, Capacitor_SMD:C_0805_2012Metric, F.Cu at (-240.5, -44.5)
- added C45: 100n, >230Vac, Capacitor_THT:C_Rect_L13.0mm_W5.0mm_P10.00mm_FKS3_FKP3_MKS4, F.Cu at (32.3, 52.6)
- added C46: 100n, >230AC, Capacitor_THT:C_Rect_L18.0mm_W6.0mm_P15.00mm_FKS3_FKP3, F.Cu at (35.6, 74.8)
- added C47: 2n2, Capacitor_THT:C_Rect_L18.0mm_W6.0mm_P15.00mm_FKS3_FKP3, F.Cu at (46.9, 105.7)
- added C48: 2n2, Capacitor_THT:C_Rect_L18.0mm_W6.0mm_P15.00mm_FKS3_FKP3, F.Cu at (52.3, 82.9)
- added C49: 100n, >230Vac, Capacitor_THT:C_Rect_L13.0mm_W5.0mm_P10.00mm_FKS3_FKP3_MKS4, F.Cu at (34.5, 110.8)
- added C5: 680u, Capacitor_THT:CP_Radial_D35.0mm_P10.00mm_SnapIn, F.Cu at (72.6, 49.8)
- added C50: 100n, >230Vac, Capacitor_THT:C_Rect_L13.0mm_W5.0mm_P10.00mm_FKS3_FKP3_MKS4, F.Cu at (34.5, 124.5)
- added C51: 10n, 1kV, Capacitor_SMD:C_1206_3216Metric, F.Cu at (-320.8, -37.4)
- added C52: 100n, 50V, Capacitor_SMD:C_0603_1608Metric, F.Cu at (-282.1, -75.6)
- added C53: 10u, 50V, Capacitor_THT:CP_Radial_D5.0mm_P2.00mm, F.Cu at (-327.9, -35.8)
- added C54: 2n2, 250VAC, Capacitor_THT:C_Rect_L18.0mm_W6.0mm_P15.00mm_FKS3_FKP3, F.Cu at (-302.9, -80.6)
- added C55: 470u, Capacitor_THT:C_Radial_D10.0mm_H16.0mm_P5.00mm, F.Cu at (-298.6, -56.5)
- added C56: 470u, Capacitor_THT:C_Radial_D10.0mm_H16.0mm_P5.00mm, F.Cu at (-298.6, -45.0)
- added C57: 2n2, Capacitor_THT:C_Rect_L18.0mm_W6.0mm_P15.00mm_FKS3_FKP3, F.Cu at (-319.9, -100.4)
- added C58: 4u7, 20V, Capacitor_SMD:C_0805_2012Metric, F.Cu at (-313.0, -60.8)
- added C59: 10u, Capacitor_SMD:C_0805_2012Metric, F.Cu at (-313.0, -57.8)
- added C60: 22u, Capacitor_SMD:C_0805_2012Metric, F.Cu at (-313.0, -54.8)
- added C61: 100n, 16V, Capacitor_SMD:C_0805_2012Metric, F.Cu at (-308.5, -60.8)
- added C62: 47u, Capacitor_SMD:C_1206_3216Metric, F.Cu at (-320.8, -34.1)
- added C63: 1u, Capacitor_SMD:C_0805_2012Metric, F.Cu at (-308.5, -57.8)
- added C64: 10u, Capacitor_SMD:C_0805_2012Metric, F.Cu at (-308.5, -54.8)
- added C65: 1u, Capacitor_SMD:C_0805_2012Metric, F.Cu at (-304.1, -60.8)
- added C66: 1u, Capacitor_SMD:C_0805_2012Metric, F.Cu at (-304.1, -57.8)
- added C67: 22u, Capacitor_SMD:C_0805_2012Metric, F.Cu at (-304.1, -54.8)
- added C68: 100n, Capacitor_SMD:C_0805_2012Metric, F.Cu at (-205.4, -67.3)
- added C69: 100n, Capacitor_SMD:C_0805_2012Metric, F.Cu at (-205.4, -64.3)
- added C70: 100n, Capacitor_SMD:C_0805_2012Metric, F.Cu at (-205.4, -61.2)
- added C71: 100n, Capacitor_SMD:C_0805_2012Metric, F.Cu at (-200.9, -67.3)
- added C72: 4u7, Capacitor_SMD:C_0805_2012Metric, F.Cu at (-200.9, -64.3)
- added C73: 27p, Capacitor_SMD:C_0603_1608Metric, F.Cu at (-224.7, -67.0)
- added C74: 27p, Capacitor_SMD:C_0603_1608Metric, F.Cu at (-224.7, -64.5)
- added C75: 100n, Capacitor_SMD:C_0805_2012Metric, F.Cu at (-200.9, -61.2)
- added C76: 100n, Capacitor_SMD:C_0805_2012Metric, F.Cu at (-196.5, -67.3)
- added C77: 100n, Capacitor_SMD:C_0805_2012Metric, F.Cu at (-196.5, -64.3)
- added C78: 100n, Capacitor_SMD:C_0805_2012Metric, F.Cu at (-196.5, -61.2)
- added C79: 100n, Capacitor_SMD:C_0805_2012Metric, F.Cu at (-216.8, -190.6)
- added C80: 1u, Capacitor_SMD:C_0805_2012Metric, F.Cu at (-216.8, -187.6)
- added C81: 1u, Capacitor_SMD:C_0805_2012Metric, F.Cu at (-216.8, -184.6)
- added C82: 100n, Capacitor_SMD:C_0805_2012Metric, F.Cu at (-216.8, -181.6)
- added C83: 10u, Capacitor_SMD:C_0805_2012Metric, F.Cu at (-216.8, -178.6)
- added C84: 1u, Capacitor_SMD:C_0805_2012Metric, F.Cu at (-216.8, -175.6)
- added C85: 100n, Capacitor_SMD:C_0805_2012Metric, F.Cu at (-212.3, -190.6)
- added C86: 100n, Capacitor_SMD:C_0805_2012Metric, F.Cu at (-212.3, -187.6)
- added C87: 100n, Capacitor_SMD:C_0805_2012Metric, F.Cu at (-212.3, -184.6)
- added C88: 1u, Capacitor_SMD:C_0805_2012Metric, F.Cu at (-212.3, -181.6)
- added C89: 1u, Capacitor_SMD:C_0805_2012Metric, F.Cu at (-212.3, -178.6)
- added C9: C_Small, Capacitor_SMD:C_1206_3216Metric, F.Cu at (-228.2, -117.2)
- added D1: 1N4148, Diode_THT:D_DO-35_SOD27_P7.62mm_Horizontal, F.Cu at (-37.6, -167.3)
- added D11: LED, LED_SMD:LED_1206_3216Metric, F.Cu at (-239.4, -133.7)
- added D15: LED, LED_SMD:LED_1206_3216Metric, F.Cu at (-239.4, -120.1)
- added D18: LED, LED_SMD:LED_1206_3216Metric, F.Cu at (-239.4, -110.0)
- added D19: BAT54S, Package_TO_SOT_SMD:SOT-23, F.Cu at (-253.6, -75.0)
- added D2: 1N4148, Diode_THT:D_DO-35_SOD27_P7.62mm_Horizontal, F.Cu at (-37.6, -163.8)
- added D20: BAT54S, Package_TO_SOT_SMD:SOT-23, F.Cu at (-253.6, -70.6)
- added D21: BAT54S, Package_TO_SOT_SMD:SOT-23, F.Cu at (-253.6, -66.1)
- added D22: BAT54S, Package_TO_SOT_SMD:SOT-23, F.Cu at (-253.6, -61.7)
- added D23: BAT54S, Package_TO_SOT_SMD:SOT-23, F.Cu at (-253.6, -57.2)
- added D24: BAT54S, Package_TO_SOT_SMD:SOT-23, F.Cu at (-248.7, -75.0)
- added D25: BAT54S, Package_TO_SOT_SMD:SOT-23, F.Cu at (-248.7, -70.6)
- added D26: BAT54S, Package_TO_SOT_SMD:SOT-23, F.Cu at (-248.7, -66.1)
- added D27: BAT54S, Package_TO_SOT_SMD:SOT-23, F.Cu at (-248.7, -61.7)
- added D28: BAT54S, Package_TO_SOT_SMD:SOT-23, F.Cu at (-248.7, -57.2)
- added D29: BAT54S, Package_TO_SOT_SMD:SOT-23, F.Cu at (-243.8, -75.0)
- added D30: BAT54S, Package_TO_SOT_SMD:SOT-23, F.Cu at (-243.8, -70.6)
- added D31: BAT54S, Package_TO_SOT_SMD:SOT-23, F.Cu at (-243.8, -66.1)
- added D32: BAT54S, Package_TO_SOT_SMD:SOT-23, F.Cu at (-243.8, -61.7)
- added D33: 1N4007, Diode_THT:D_DO-41_SOD81_P10.16mm_Horizontal, F.Cu at (57.5, 45.5)
- added D34: 1N4007, Diode_THT:D_DO-41_SOD81_P10.16mm_Horizontal, F.Cu at (59.4, 118.3)
- added D35: P6KE150A, Diode_THT:D_DO-15_P10.16mm_Horizontal, F.Cu at (-328.3, -45.9)
- added D36: 1N4007, Diode_THT:D_DO-41_SOD81_P10.16mm_Horizontal, F.Cu at (-328.4, -41.2)
- added D37: SB24, Diode_SMD:D_SOD-128, F.Cu at (-311.5, -39.5)
- added D38: SB24, Diode_SMD:D_SOD-128, F.Cu at (-311.5, -35.4)
- added D39: BZX79-C11, Diode_THT:D_DO-35_SOD27_P7.62mm_Horizontal, F.Cu at (-300.3, -37.4)
- added D40: SK15, Diode_SMD:D_SMA_Handsoldering, F.Cu at (-285.2, -60.0)
- added D41: SK15, Diode_SMD:D_SMA_Handsoldering, F.Cu at (-285.2, -55.5)
- added D42: TVS, Diode_SMD:D_SOD-523, F.Cu at (-220.9, -67.1)
- added D43: 1N4148, Diode_THT:D_DO-35_SOD27_P7.62mm_Horizontal, F.Cu at (-217.4, -55.6)
- added D44: 1N4148, Diode_THT:D_DO-35_SOD27_P7.62mm_Horizontal, F.Cu at (-217.4, -52.1)
- added D45: 1N4148, Diode_THT:D_DO-35_SOD27_P7.62mm_Horizontal, F.Cu at (-217.4, -48.5)
- added D7: D, Package_TO_SOT_THT:TO-220-2_Vertical, F.Cu at (148.5, -152.1)
- added D8: schottky, Package_TO_SOT_SMD:TO-263-2, F.Cu at (-279.3, -129.2)
- added D9: schottky, Package_TO_SOT_SMD:TO-263-2, F.Cu at (-279.3, -116.9)
- added F2: Polyfuse, Varistor:RV_Disc_D15.5mm_W5mm_P7.5mm, F.Cu at (-204.0, -82.2)
- added FB1: 120R, Inductor_SMD:L_0805_2012Metric, F.Cu at (-224.4, -45.1)
- added J3: USB_C_Receptacle_USB2.0_16P, Connector_USB:USB_C_Receptacle_GCT_USB4105-xx-A_16P_TopMnt_Horizontal, F.Cu at (-201.8, -54.5)
- added K2: SPST-NO, filip:Industrial-Relays-OJS-SS-112HEF_SPST-NO, F.Cu at (55.4, 126.9)
- added L2: 220u, filip:ETD-39-Inductor, F.Cu at (-283.3, -151.9)
- added L3: 2m2, filip:Common_Mode_Choke_2Line, F.Cu at (20.3, 97.9)
- added M1: Fan_4pin, Connector:FanPinHeader_1x04_P2.54mm_Vertical, F.Cu at (-228.8, -80.7)
- added M2: Fan_4pin, Connector:FanPinHeader_1x04_P2.54mm_Vertical, F.Cu at (-228.8, -72.6)
- added Q3: NMOS, Package_TO_SOT_SMD:SOT-23-3, F.Cu at (155.3, 36.1)
- added Q4: IPZA60R070CM8XKSA1, Package_TO_SOT_THT:TO-247-4_Vertical, F.Cu at (131.9, -152.8)
- added Q5: IPZA60R070CM8XKSA1, Package_TO_SOT_THT:TO-247-4_Vertical, F.Cu at (159.9, -152.8)
- added Q6: NMOS, Package_TO_SOT_SMD:SOT-23-3, F.Cu at (54.6, 58.7)
- added Q7: NMOS, Package_TO_SOT_SMD:SOT-23-3, F.Cu at (57.9, 131.8)
- added Q8: 2N7002, Package_TO_SOT_SMD:SOT-23, F.Cu at (-193.5, -57.5)
- added Q9: 2N7002, Package_TO_SOT_SMD:SOT-23, F.Cu at (-193.5, -53.1)
- added R100: 3.6M, 325V, Resistor_THT:R_Axial_DIN0309_L9.0mm_D3.2mm_P12.70mm_Horizontal, F.Cu at (-303.6, -69.3)
- added R101: 1k, Resistor_SMD:R_0805_2012Metric, F.Cu at (-286.3, -75.4)
- added R102: 100, 325V, Resistor_THT:R_Axial_DIN0411_L9.9mm_D3.6mm_P12.70mm_Horizontal, F.Cu at (-303.2, -74.3)
- added R103: 390 1/8W, Resistor_SMD:R_0805_2012Metric, F.Cu at (-286.3, -72.4)
- added R104: 2k 1/8W, Resistor_SMD:R_0805_2012Metric, F.Cu at (-286.3, -69.5)
- added R105: 34k, Resistor_SMD:R_0603_1608Metric, F.Cu at (-282.1, -73.1)
- added R106: 4k7, Resistor_SMD:R_0805_2012Metric, F.Cu at (-286.3, -66.5)
- added R107: 10k, Resistor_SMD:R_0805_2012Metric, F.Cu at (-228.9, -66.8)
- added R108: 10k, Resistor_SMD:R_0805_2012Metric, F.Cu at (-228.9, -63.9)
- added R109: 5k1, Resistor_SMD:R_0805_2012Metric, F.Cu at (-228.9, -60.9)
- added R11: 4k7, Resistor_SMD:R_0805_2012Metric, F.Cu at (-118.6, -109.1)
- added R110: 5k1, Resistor_SMD:R_0805_2012Metric, F.Cu at (-228.9, -58.0)
- added R111: 22, Resistor_SMD:R_0603_1608Metric, F.Cu at (-224.7, -62.0)
- added R112: 22, Resistor_SMD:R_0603_1608Metric, F.Cu at (-224.7, -59.5)
- added R113: 1k5, Resistor_SMD:R_0603_1608Metric, F.Cu at (-224.7, -57.0)
- added R114: 10k, Resistor_SMD:R_0805_2012Metric, F.Cu at (-228.9, -55.0)
- added R115: 10k, Resistor_SMD:R_0805_2012Metric, F.Cu at (-228.9, -52.1)
- added R116: 10k, Resistor_SMD:R_0805_2012Metric, F.Cu at (-228.9, -49.1)
- added R117: 10k, Resistor_SMD:R_0805_2012Metric, F.Cu at (-228.9, -46.2)
- added R118: R_Small, Resistor_SMD:R_0603_1608Metric, F.Cu at (-208.1, -190.8)
- added R119: R_Small, Resistor_SMD:R_0603_1608Metric, F.Cu at (-208.1, -188.3)
- added R120: 1k, Resistor_SMD:R_0805_2012Metric, F.Cu at (-216.8, -166.7)
- added R121: 100k, Resistor_SMD:R_0805_2012Metric, F.Cu at (-216.8, -163.8)
- added R122: R_Small, Resistor_SMD:R_0603_1608Metric, F.Cu at (-208.1, -185.8)
- added R123: R_Small, Resistor_SMD:R_0603_1608Metric, F.Cu at (-208.1, -183.3)
- added R124: R_Small, Resistor_SMD:R_0603_1608Metric, F.Cu at (-208.1, -180.8)
- added R125: R_Small, Resistor_SMD:R_0603_1608Metric, F.Cu at (-208.1, -178.3)
- added R126: 1k, Resistor_SMD:R_0805_2012Metric, F.Cu at (-216.8, -160.8)
- added R16: 0, Resistor_SMD:R_0603_1608Metric, F.Cu at (159.8, 48.3)
- added R19: 3, 1W, Resistor_SMD:R_1206_3216Metric, F.Cu at (143.6, -148.6)
- added R20: 3, 1W, Resistor_SMD:R_1206_3216Metric, F.Cu at (168.8, -148.3)
- added R21: 10m, Resistor_SMD:R_0805_2012Metric, F.Cu at (-503.1, -111.3)
- added R22: R_Small, Resistor_SMD:R_1206_3216Metric, F.Cu at (-233.8, -123.8)
- added R23: R_Small, Resistor_SMD:R_1206_3216Metric, F.Cu at (-233.8, -120.5)
- added R25: 5k1, Resistor_SMD:R_0805_2012Metric, F.Cu at (-316.7, -120.3)
- added R26: 5k1, Resistor_SMD:R_0805_2012Metric, F.Cu at (-316.7, -117.3)
- added R27: 5k1, Resistor_SMD:R_0805_2012Metric, F.Cu at (-316.7, -114.4)
- added R28: 5k1, Resistor_SMD:R_0805_2012Metric, F.Cu at (-316.7, -111.4)
- added R31: 5k1, Resistor_SMD:R_0805_2012Metric, F.Cu at (-312.3, -123.2)
- added R34: 10k, 1W, Resistor_SMD:R_2512_6332Metric, F.Cu at (-233.8, -110.6)
- added R35: 10k, 1W, Resistor_SMD:R_2512_6332Metric, F.Cu at (-205.5, -164.4)
- added R36: 10k, 1W, Resistor_SMD:R_2512_6332Metric, F.Cu at (-205.5, -159.5)
- added R37: 10k, 1W, Resistor_SMD:R_2512_6332Metric, F.Cu at (-205.5, -154.6)
- added R38: 10k, 1W, Resistor_SMD:R_2512_6332Metric, F.Cu at (-205.5, -149.7)
- added R47: 3k3, Resistor_SMD:R_0805_2012Metric, F.Cu at (-275.9, -52.2)
- added R48: 3k3, Resistor_SMD:R_0805_2012Metric, F.Cu at (-275.9, -49.2)
- added R49: 1k, Resistor_SMD:R_0805_2012Metric, F.Cu at (-271.5, -75.8)
- added R5: 330, Resistor_SMD:R_0805_2012Metric, F.Cu at (-325.5, -117.3)
- added R50: 1k, Resistor_SMD:R_0805_2012Metric, F.Cu at (-271.5, -72.8)
- added R51: 1k, Resistor_SMD:R_0805_2012Metric, F.Cu at (-271.5, -69.9)
- added R52: 1k, Resistor_SMD:R_0805_2012Metric, F.Cu at (-271.5, -66.9)
- added R53: 1k, Resistor_SMD:R_0805_2012Metric, F.Cu at (-271.5, -64.0)
- added R54: 1k, Resistor_SMD:R_0805_2012Metric, F.Cu at (-271.5, -61.0)
- added R55: 3k3, Resistor_SMD:R_0805_2012Metric, F.Cu at (-271.5, -58.1)
- added R56: 3k3, Resistor_SMD:R_0805_2012Metric, F.Cu at (-271.5, -55.1)
- added R57: 3k3, Resistor_SMD:R_0805_2012Metric, F.Cu at (-271.5, -52.2)
- added R58: 3k3, Resistor_SMD:R_0805_2012Metric, F.Cu at (-271.5, -49.2)
- added R59: 3k3, Resistor_SMD:R_0805_2012Metric, F.Cu at (-267.1, -75.8)
- added R60: 27k, Resistor_SMD:R_0805_2012Metric, F.Cu at (-267.1, -72.8)
- added R61: 27k, Resistor_SMD:R_0805_2012Metric, F.Cu at (-267.1, -69.9)
- added R62: 27k, Resistor_SMD:R_0805_2012Metric, F.Cu at (-267.1, -66.9)
- added R63: 3k3, Resistor_SMD:R_0805_2012Metric, F.Cu at (-267.1, -64.0)
- added R64: 3k3, Resistor_SMD:R_0805_2012Metric, F.Cu at (-267.1, -61.0)
- added R65: 3k3, Resistor_SMD:R_0805_2012Metric, F.Cu at (-267.1, -58.1)
- added R66: 3k3, Resistor_SMD:R_0805_2012Metric, F.Cu at (-267.1, -55.1)
- added R67: 3k3, Resistor_SMD:R_0805_2012Metric, F.Cu at (-267.1, -52.2)
- added R68: 10k, Resistor_SMD:R_0805_2012Metric, F.Cu at (-267.1, -49.2)
- added R69: 10k, Resistor_SMD:R_0805_2012Metric, F.Cu at (-262.7, -75.8)
- added R7: 1k, Resistor_SMD:R_0805_2012Metric, F.Cu at (-325.5, -111.4)
- added R70: 3k3, Resistor_SMD:R_0805_2012Metric, F.Cu at (-262.7, -72.8)
- added R71: 3k3, Resistor_SMD:R_0805_2012Metric, F.Cu at (-262.7, -69.9)
- added R72: 3k3, Resistor_SMD:R_0805_2012Metric, F.Cu at (-262.7, -66.9)
- added R73: 22k, Resistor_SMD:R_0603_1608Metric, F.Cu at (-235.3, -73.5)
- added R74: 3k3, Resistor_SMD:R_0805_2012Metric, F.Cu at (-262.7, -64.0)
- added R75: 22k, Resistor_SMD:R_0603_1608Metric, F.Cu at (-235.3, -71.0)
- added R76: 1k, Resistor_SMD:R_0805_2012Metric, F.Cu at (-262.7, -61.0)
- added R77: 3k3, Resistor_SMD:R_0805_2012Metric, F.Cu at (-262.7, -58.1)
- added R78: 3k3, Resistor_SMD:R_0805_2012Metric, F.Cu at (-262.7, -55.1)
- added R79: 68k, Resistor_SMD:R_0805_2012Metric, F.Cu at (-262.7, -52.2)
- added R8: 1k, Resistor_SMD:R_0805_2012Metric, F.Cu at (-321.1, -129.1)
- added R80: 68k, Resistor_SMD:R_0805_2012Metric, F.Cu at (-262.7, -49.2)
- added R81: 68k, Resistor_SMD:R_0805_2012Metric, F.Cu at (-258.3, -75.8)
- added R82: 68k, Resistor_SMD:R_0805_2012Metric, F.Cu at (-258.3, -72.8)
- added R83: 68k, Resistor_SMD:R_0805_2012Metric, F.Cu at (-258.3, -69.9)
- added R84: R_Small, Resistor_SMD:R_0603_1608Metric, F.Cu at (-235.3, -68.5)
- added R85: 27k, Resistor_SMD:R_0805_2012Metric, F.Cu at (-258.3, -66.9)
- added R86: 27k, Resistor_SMD:R_0805_2012Metric, F.Cu at (-258.3, -64.0)
- added R87: 27k, Resistor_SMD:R_0805_2012Metric, F.Cu at (-258.3, -61.0)
- added R88: 3k3, Resistor_SMD:R_0805_2012Metric, F.Cu at (-258.3, -58.1)
- added R89: 3k3, Resistor_SMD:R_0805_2012Metric, F.Cu at (-258.3, -55.1)
- added R9: 1k, Resistor_SMD:R_0805_2012Metric, F.Cu at (-321.1, -126.2)
- added R90: 3k3, Resistor_SMD:R_0805_2012Metric, F.Cu at (-258.3, -52.2)
- added R91: 22, Resistor_SMD:R_1206_3216Metric, F.Cu at (55.5, 42.9)
- added R92: 1k, Resistor_SMD:R_0805_2012Metric, F.Cu at (57.9, 61.5)
- added R93: 10k, Resistor_SMD:R_0805_2012Metric, F.Cu at (54.5, 61.5)
- added R94: 100, >230Vac, Resistor_THT:R_Axial_DIN0411_L9.9mm_D3.6mm_P12.70mm_Horizontal, F.Cu at (36.6, 59.9)
- added R95: 22, Resistor_SMD:R_1206_3216Metric, F.Cu at (57.7, 115.8)
- added R96: 27, filip:Resistor_THT_Power_Axial_WW20W_P27mm, F.Cu at (22.0, 120.4)
- added R97: 1k, Resistor_SMD:R_0805_2012Metric, F.Cu at (61.2, 134.6)
- added R98: 10k, Resistor_SMD:R_0805_2012Metric, F.Cu at (57.7, 134.6)
- added R99: 100, >230Vac, Resistor_THT:R_Axial_DIN0411_L9.9mm_D3.6mm_P12.70mm_Horizontal, F.Cu at (38.9, 134.3)
- added RV1: Varistor, Varistor:RV_Disc_D15.5mm_W5mm_P7.5mm, F.Cu at (31.7, 69.9)
- added RV2: 100k, filip:Potentiometer_SMD_Trimmer_PVG3_3.6x3, F.Cu at (-216.6, -171.4)
- added RV3: 100k, filip:Potentiometer_SMD_Trimmer_PVG3_3.6x3, F.Cu at (-211.8, -171.4)
- added TH1: 10k, Connector_PinHeader_2.54mm:PinHeader_1x02_P2.54mm_Vertical, F.Cu at (-275.8, -82.1)
- added TH2: 10k, Connector_PinHeader_2.54mm:PinHeader_1x02_P2.54mm_Vertical, F.Cu at (-271.2, -82.1)
- added TH3: 10k, Connector_PinHeader_2.54mm:PinHeader_1x02_P2.54mm_Vertical, F.Cu at (-266.6, -82.1)
- added TH4: 10k, Connector_PinHeader_2.54mm:PinHeader_1x02_P2.54mm_Vertical, F.Cu at (-262.0, -82.1)
- added TH5: 10k, Connector_PinHeader_2.54mm:PinHeader_1x02_P2.54mm_Vertical, F.Cu at (-257.5, -82.1)
- added TH6: 10k, Resistor_SMD:R_0603_1608Metric, F.Cu at (-235.3, -66.0)
- added TH7: 10k, Connector_PinHeader_2.54mm:PinHeader_1x02_P2.54mm_Vertical, F.Cu at (-252.9, -82.1)
- added TH8: 10k, Connector_PinHeader_2.54mm:PinHeader_1x02_P2.54mm_Vertical, F.Cu at (-248.3, -82.1)
- added TH9: 10k, Connector_PinHeader_2.54mm:PinHeader_1x02_P2.54mm_Vertical, F.Cu at (-243.7, -82.1)
- added TP1: LIVE_IN, Connector_Pin:Pin_D0.7mm_L6.5mm_W1.8mm_FlatFork, F.Cu at (17.5, 34.6)
- added TP10: HS, Connector_Pin:Pin_D0.7mm_L6.5mm_W1.8mm_FlatFork, F.Cu at (-22.8, 26.7)
- added TP11: LS, Connector_Pin:Pin_D0.7mm_L6.5mm_W1.8mm_FlatFork, F.Cu at (-22.8, 30.1)
- added TP12: +RECT, Connector_Pin:Pin_D0.7mm_L6.5mm_W1.8mm_FlatFork, F.Cu at (-22.8, 33.6)
- added TP13: -RECT, Connector_Pin:Pin_D0.7mm_L6.5mm_W1.8mm_FlatFork, F.Cu at (-19.0, 23.2)
- added TP14: +70V, Connector_Pin:Pin_D0.7mm_L6.5mm_W1.8mm_FlatFork, F.Cu at (-19.0, 26.7)
- added TP15: -70V, Connector_Pin:Pin_D0.7mm_L6.5mm_W1.8mm_FlatFork, F.Cu at (-19.0, 30.1)
- added TP16: PRIM_SHUNT_H, Connector_Pin:Pin_D0.7mm_L6.5mm_W1.8mm_FlatFork, F.Cu at (-13.2, 23.2)
- added TP17: PRIM_SHUNT_L, Connector_Pin:Pin_D0.7mm_L6.5mm_W1.8mm_FlatFork, F.Cu at (-13.2, 26.7)
- added TP2: NEUTRAL_IN, Connector_Pin:Pin_D0.7mm_L6.5mm_W1.8mm_FlatFork, F.Cu at (24.2, 34.6)
- added TP3: LIVE_OUT, Connector_Pin:Pin_D0.7mm_L6.5mm_W1.8mm_FlatFork, F.Cu at (72.7, 139.6)
- added TP4: NEUTRAL_OUT, Connector_Pin:Pin_D0.7mm_L6.5mm_W1.8mm_FlatFork, F.Cu at (58.2, 105.0)
- added TP5: HG, Connector_Pin:Pin_D0.7mm_L6.5mm_W1.8mm_FlatFork, F.Cu at (-26.6, 23.2)
- added TP6: VBUS, Connector_Pin:Pin_D0.7mm_L6.5mm_W1.8mm_FlatFork, F.Cu at (-26.6, 26.7)
- added TP7: LG, Connector_Pin:Pin_D0.7mm_L6.5mm_W1.8mm_FlatFork, F.Cu at (-26.6, 30.1)
- added TP8: HP, Connector_Pin:Pin_D0.7mm_L6.5mm_W1.8mm_FlatFork, F.Cu at (-26.6, 33.6)
- added TP9: LP, Connector_Pin:Pin_D0.7mm_L6.5mm_W1.8mm_FlatFork, F.Cu at (-22.8, 23.2)
- added U13: AMC1350DWV, Package_SO:SOIC-8_7.5x5.85mm_P1.27mm, F.Cu at (-271.1, -44.0)
- added U14: LM358, Package_SO:TSSOP-8_3x3mm_P0.65mm, F.Cu at (-237.9, -62.4)
- added U16: TNY274P, Package_DIP:PowerIntegrations_PDIP-8C, F.Cu at (-313.2, -51.2)
- added U17: PC817, Package_SO:SOP-4_4.4x2.6mm_P1.27mm, F.Cu at (-285.5, -34.4)
- added U18: 5V LDO, Package_TO_SOT_SMD:SOT-223-3_TabPin2, F.Cu at (-285.4, -49.0)
- added U19: LMR51430, Package_TO_SOT_SMD:SOT-23-6, F.Cu at (-305.2, -39.1)
- added U2: ISO6720BD, Package_SO:SOIC-8_3.9x4.9mm_P1.27mm, F.Cu at (-237.5, -150.3)
- added U20: TPS60403DBV, Package_TO_SOT_SMD:SOT-23-5, F.Cu at (-305.2, -34.5)
- added U21: 3v3 LDO, Package_TO_SOT_SMD:SOT-223-3_TabPin2, F.Cu at (-285.4, -40.7)
- added U22: USBLC6-2SC6, Package_TO_SOT_SMD:SOT-23-6, F.Cu at (-224.1, -53.3)
- added U23: STM32F103C8Tx, Package_QFP:LQFP-48_7x7mm_P0.5mm, F.Cu at (-213.3, -63.1)
- added U24: TPS3823-xxDBV, Package_TO_SOT_SMD:SOT-23-5, F.Cu at (-224.1, -48.7)
- added U25: LMV393, Package_SO:SOIC-8_3.9x4.9mm_P1.27mm, F.Cu at (-223.2, -182.2)
- added U25: LMV393, Package_SO:SOIC-8_3.9x4.9mm_P1.27mm, F.Cu at (-223.2, -188.7)
- added U26: NE555D, Package_SO:SOIC-8_3.9x4.9mm_P1.27mm, F.Cu at (-223.2, -175.6)
- added U27: LMV393, Package_SO:SOIC-8_3.9x4.9mm_P1.27mm, F.Cu at (-223.2, -169.0)
- added U28: LMV393, Package_SO:SOIC-8_3.9x4.9mm_P1.27mm, F.Cu at (-223.2, -162.4)
- added Y1: 8MHz, filip:HC-49US, F.Cu at (-200.2, -74.9)
- C1: value 680u -> 100n; footprint Capacitor_THT:CP_Radial_D35.0mm_P10.00mm_SnapIn -> Capacitor_SMD:C_0805_2012Metric
- C12: value 2n2, 250VAC -> 2m2; footprint Capacitor_THT:C_Rect_L18.0mm_W6.0mm_P15.00mm_FKS3_FKP3 -> Capacitor_THT:CP_Radial_D30.0mm_P10.00mm_SnapIn
- C17: value 680u -> 2m2; footprint Capacitor_THT:CP_Radial_D35.0mm_P10.00mm_SnapIn -> Capacitor_THT:CP_Radial_D30.0mm_P10.00mm_SnapIn
- C20: value 100n -> 2m2; footprint Capacitor_SMD:C_0805_2012Metric -> Capacitor_THT:CP_Radial_D30.0mm_P10.00mm_SnapIn
- C22: value 10u -> 1u
- C23: value 22u -> 1u
- C24: value 100n, 16V -> TBD; footprint Capacitor_SMD:C_0805_2012Metric -> Capacitor_SMD:C_0603_1608Metric
- C26: value 10u -> TBD; footprint Capacitor_SMD:C_0805_2012Metric -> Capacitor_SMD:C_0603_1608Metric
- C27: value 22u -> TBD; footprint Capacitor_SMD:C_0805_2012Metric -> Capacitor_SMD:C_0603_1608Metric
- C28, C29: value 2m2 -> 100n; footprint Capacitor_THT:CP_Radial_D30.0mm_P10.00mm_SnapIn -> Capacitor_SMD:C_0805_2012Metric
- C3: value 2m2 -> 680u; footprint Capacitor_THT:CP_Radial_D30.0mm_P10.00mm_SnapIn -> Capacitor_THT:CP_Radial_D35.0mm_P10.00mm_SnapIn
- C30, C31, C32, C33: value 2m2 -> 1u; footprint Capacitor_THT:CP_Radial_D30.0mm_P10.00mm_SnapIn -> Capacitor_SMD:C_0805_2012Metric
- C36, C37: value 100n -> 1u
- C39: value 4u7 -> 300p; footprint Capacitor_SMD:C_0805_2012Metric -> Capacitor_SMD:C_0603_1608Metric
- C40: value 100n -> 300p; footprint Capacitor_SMD:C_0805_2012Metric -> Capacitor_SMD:C_0603_1608Metric
- C44: value 100n -> 100n, >230Vac; footprint Capacitor_SMD:C_0805_2012Metric -> Capacitor_THT:C_Rect_L13.0mm_W5.0mm_P10.00mm_FKS3_FKP3_MKS4
- C6: footprint Capacitor_THT:C_Rect_L18.0mm_W6.0mm_P15.00mm_FKS3_FKP3 -> Capacitor_SMD:C_0805_2012Metric
- C7: value 2n2 -> 100n; footprint Capacitor_THT:C_Rect_L18.0mm_W6.0mm_P15.00mm_FKS3_FKP3 -> Capacitor_SMD:C_0805_2012Metric
- C8: value 2n2 -> C_Small; footprint Capacitor_THT:C_Rect_L18.0mm_W6.0mm_P15.00mm_FKS3_FKP3 -> Capacitor_SMD:C_1206_3216Metric
- D10: value 1N4007 -> schottky; footprint Diode_THT:D_DO-41_SOD81_P10.16mm_Horizontal -> Package_TO_SOT_SMD:TO-263-2
- D12: value 1N4007 -> LED; footprint Diode_THT:D_DO-41_SOD81_P10.16mm_Horizontal -> LED_SMD:LED_1206_3216Metric
- D13, D14: value D_Schottky -> LED; footprint Diode_SMD:D_1206_3216Metric -> LED_SMD:LED_1206_3216Metric
- D16, D17: value BYG20J -> LED; footprint Diode_SMD:D_SMA -> LED_SMD:LED_1206_3216Metric
- D4, D5: value schottky -> BYG20J; footprint Package_TO_SOT_SMD:TO-263-2 -> Diode_SMD:D_SMA
- D6: value schottky -> D; footprint Package_TO_SOT_SMD:TO-263-2 -> Package_TO_SOT_THT:TO-220-2_Vertical
- J2: value Conn_ARM_JTAG_SWD_10 -> Conn_02x07_Odd_Even; footprint Connector_PinHeader_1.27mm:PinHeader_2x05_P1.27mm_Vertical_SMD -> Connector_PinHeader_2.54mm:PinHeader_2x07_P2.54mm_Vertical_SMD
- J4: value Conn_01x04_Pin -> Conn_ARM_JTAG_SWD_10; footprint Connector_JST:JST_EH_S4B-EH_1x04_P2.50mm_Horizontal -> Connector_PinHeader_1.27mm:PinHeader_2x05_P1.27mm_Vertical_SMD
- L1: value 2m2 -> 220u; footprint filip:Common_Mode_Choke_2Line -> filip:ETD-39-Inductor
- Q1: value IPZA60R070CM8XKSA1 -> NPN; footprint Package_TO_SOT_THT:TO-247-4_Vertical -> Package_TO_SOT_SMD:SOT-23
- Q2: value IPZA60R070CM8XKSA1 -> NMOS; footprint Package_TO_SOT_THT:TO-247-4_Vertical -> Package_TO_SOT_SMD:SOT-223-3_TabPin2
- R1: value 22 -> 330; footprint Resistor_SMD:R_1206_3216Metric -> Resistor_SMD:R_0805_2012Metric
- R10: value 3k3 -> 1k
- R12: value 10k -> 100k
- R13: value 10k -> 5
- R14: value 3.6M -> 2.2; footprint Resistor_SMD:R_0805_2012Metric -> Resistor_SMD:R_1206_3216Metric
- R15: value 1k -> 0; footprint Resistor_SMD:R_0805_2012Metric -> Resistor_SMD:R_0603_1608Metric
- R17: value 390 1/8W -> 470
- R18: value 2k 1/8W -> 470
- R2: value 27 -> 330; footprint filip:Resistor_THT_Power_Axial_WW20W_P27mm -> Resistor_SMD:R_0805_2012Metric
- R24: value 10k -> 5k1
- R29: value 34k -> 5k1
- R3: value 1k -> 330
- R30: value 4k7 -> 5k1
- R32: value 10k -> 15m
- R33: value 10k -> 10k, 1W; footprint Resistor_SMD:R_1206_3216Metric -> Resistor_SMD:R_2512_6332Metric
- R39, R40, R45, R46: value 5k1 -> 3k3
- R4: value 10k -> 330
- R41, R42, R43, R44: value 5k1 -> 100
- R6: value 4k7 -> 1k
- U1: value UCC27714D -> LTV-847S; footprint Package_SO:SOIC-14_3.9x8.7mm_P1.27mm -> Package_DIP:SMDIP-16_W9.53mm
- U10: value PC837 -> INA180A2; footprint Package_DIP:DIP-12_W7.62mm -> Package_TO_SOT_SMD:SOT-23-5
- U11: value B66398W1024T1 -> INA180A1; footprint filip:ETD59 -> Package_TO_SOT_SMD:SOT-23-5
- U12: value STM32F103C8Tx -> AMC1350; footprint Package_QFP:LQFP-48_7x7mm_P0.5mm -> Package_TO_SOT_SMD:SOT-23-6
- U15: value USBLC6-2SC6 -> TLV6001DCK; footprint Package_TO_SOT_SMD:SOT-23-6 -> Package_TO_SOT_SMD:SOT-353_SC-70-5
- U3: value INA180A4 -> LTV-827S; footprint Package_TO_SOT_SMD:SOT-23-5 -> Package_DIP:SMDIP-8_W9.53mm
- U4: value PC837 -> UCC27714D; footprint Package_DIP:DIP-12_W7.62mm -> Package_SO:SOIC-14_3.9x8.7mm_P1.27mm
- U5: value TNY274P -> ETD59; footprint Package_DIP:PowerIntegrations_PDIP-8C -> filip:ETD59
- U6: value PC817 -> 74HC595; footprint Package_DIP:DIP-4_W7.62mm -> Package_SO:SOIC-16_3.9x9.9mm_P1.27mm
- U7: value 5V LDO -> 74HC595; footprint Package_TO_SOT_SMD:SOT-223-3_TabPin2 -> Package_SO:SOIC-16_3.9x9.9mm_P1.27mm
- U8: value LMR51430 -> NMUX1308PW; footprint Package_TO_SOT_SMD:SOT-23-6 -> Package_SO:TSSOP-16_4.4x5mm_P0.65mm
- U9: value 3v3 LDO -> NMUX1308PW; footprint Package_TO_SOT_SMD:SOT-223-3_TabPin2 -> Package_SO:TSSOP-16_4.4x5mm_P0.65mm
- moved C12 640.3 mm to (-390.4, -176.3)
- moved R29 549.5 mm to (-312.3, -129.1)
- moved R30 549.5 mm to (-312.3, -126.2)
- moved C20 543.7 mm to (-357.9, -81.7)
- moved L4 532.4 mm to (-322.7, -55.4)
- moved T1 528.0 mm to (-326.6, -79.1)
- moved U11 527.5 mm to (-235.7, -48.0)
- moved J2 525.3 mm to (-303.7, -120.7)
- moved R1 519.2 mm to (-325.5, -129.1)
- moved R2 505.5 mm to (-325.5, -126.2)
- moved U3 498.1 mm to (-283.5, -92.5)
- moved U7 496.1 mm to (-259.7, -99.2)
- moved R3 494.2 mm to (-325.5, -123.2)
- moved R4 494.2 mm to (-325.5, -120.3)
- moved L1 492.9 mm to (-331.0, -151.9)
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Connections:
- C1 pad 1: VBUS -> Net-(U4-VDD)
- C1 pad 2: GND1 -> PRIM_SGND
- C11 pad 1: +5V -> +3V3_Secondary
- C11 pad 2: PRIM_SGND -> SEC_SGND
- C12 pad 1: VBUS -> +70V
- C12 pad 2: PRIM_SGND -> SEC_SHUNT_H
- C17 pad 1: VBUS -> SEC_SHUNT_H
- C17 pad 2: GND1 -> -70V
- C18 pad 2: Net-(C100-Pad2) -> SEC_SHUNT_H
- C19 pad 1: Net-(C100-Pad2) -> SEC_SHUNT_H
- C2 pad 1: /VREF -> Net-(U4-VDD)
- C20 pad 1: +3V3_Secondary -> +70V
- C20 pad 2: SEC_SGND -> SEC_SHUNT_H
- C22 pad 1: +12V_Secondary -> Net-(C22-Pad1)
- C22 pad 2: PRIM_SGND -> SEC_SGND
- C23 pad 1: +5V_Primary -> Net-(C23-Pad1)
- C23 pad 2: PRIM_SGND -> SEC_SGND
- C24 pad 1: /Startup Power/BOOTSTRAP -> Net-(U10-+)
- C24 pad 2: /Startup Power/SW -> PRIM_SGND
- C26 pad 1: +5V_Secondary -> Net-(U10--)
- C26 pad 2: SEC_SGND -> PRIM_SGND
- C27 pad 1: +3V3_Secondary -> /Current Sensing/-
- C28 pad 1: +70V -> +5V_Primary
- C28 pad 2: Net-(C100-Pad2) -> PRIM_SGND
- C29 pad 1: Net-(C100-Pad2) -> +3V3_Secondary
- C29 pad 2: -70V -> SEC_SGND
- C3 pad 1: Net-(C100-Pad2) -> VBUS
- C3 pad 2: -70V -> GND1
- C30 pad 1: +70V -> Net-(C30-Pad1)
- C30 pad 2: Net-(C100-Pad2) -> SEC_SGND
- C31 pad 1: Net-(C100-Pad2) -> Net-(C31-Pad1)
- C31 pad 2: -70V -> SEC_SGND
- C32 pad 1: +70V -> Net-(C32-Pad1)
- C32 pad 2: Net-(C100-Pad2) -> SEC_SGND
- C33 pad 1: Net-(C100-Pad2) -> Net-(C33-Pad1)
- C33 pad 2: -70V -> SEC_SGND
- C36 pad 1: +3V3_Secondary -> Net-(C36-Pad1)
- C37 pad 1: +3V3_Secondary -> Net-(C37-Pad1)
- C38 pad 1: +3V3_Secondary -> -5V
- C39 pad 1: +3V3_Secondary -> Net-(U15--)
- C40 pad 1: /MCU/~{RST} -> /Current Sensing/MUX_OUT
- C40 pad 2: SEC_SGND -> Net-(U15-+)
- C44 pad 1: +3V3_Secondary -> /Input Filter And Slow Start/AC_L_FUSED
- C44 pad 2: SEC_SGND -> /Input Filter And Slow Start/AC_RELAY1_RC_SNUBBER_1
- C6 pad 1: Net-(C6-Pad1) -> +3V3_Secondary
- C6 pad 2: /AC_N -> SEC_SGND
- C7 pad 1: /Input Filter And Slow Start/L_FILTERED -> +3V3_Secondary
- C7 pad 2: Earth_Protective -> SEC_SGND
- C8 pad 1: /Input Filter And Slow Start/AC_N_OUT -> /SEC_PRIM
- C8 pad 2: Earth_Protective -> /POS_SNUB
- D10 pad 1: +12V -> /NEG_RECTIFIED
- D10 pad 2: Net-(D10-A) -> /POS_RECTIFIED
- D12 pad 1: Net-(D12-K) -> SEC_SGND
- D13 pad 1: +12V_Primary -> SEC_SGND
- D14 pad 1: +12V_Secondary -> SEC_SGND
- D16 pad 1: Net-(D16-K) -> SEC_SGND
- D17 pad 1: Net-(D17-K) -> SEC_SGND
- D17 pad 2: /HS -> Net-(D17-A)
- D4 pad 1: Net-(D4A-A) -> Net-(D4-K)
- D4 pad 2: Net-(D4A-K) -> Net-(D4-A)
- D5 pad 1: Net-(D4B-A) -> Net-(D5-K)
- D5 pad 2: Net-(D4A-K) -> /HS
- D6 pad 1: GND2 -> /H_SW_NODE
- D6 pad 2: Net-(D4A-K) -> GND1
- F1 pad 2: Net-(C6-Pad1) -> /Input Filter And Slow Start/AC_L_FUSED
- J2 pad 1: +3V3_Secondary -> /Y1
- J2 pad 10: /MCU/~{RST} -> SEC_SGND
- J2 pad 2: /MCU/SWDIO -> SEC_SGND
- J2 pad 3: SEC_SGND -> /Y2
- J2 pad 4: /MCU/SWCLK -> SEC_SGND
- J2 pad 5: SEC_SGND -> /Y3
- J2 pad 6: unconnected-(J2-SWO/TDO-Pad6) -> SEC_SGND
- J2 pad 7: unconnected-(J2-KEY-Pad7) -> /Y4
- J2 pad 8: unconnected-(J2-NC/TDI-Pad8) -> SEC_SGND
- J2 pad 9: SEC_SGND -> /Y5
- J4 pad 1: /MCU/~{SS} -> +3V3_Secondary
- J4 pad 2: /MCU/SCK -> /MCU/SWDIO
- J4 pad 3: /MCU/MISO -> SEC_SGND
- J4 pad 4: /MCU/MOSI -> /MCU/SWCLK
- K1 pad 1: Net-(D10-A) -> /Input Filter And Slow Start/RELAY_SWITCH_D
- K1 pad 2: Net-(K1-COIL_2) -> /Input Filter And Slow Start/RELAY1_COIL_2
- K1 pad 3: /Input Filter And Slow Start/L_FILTERED -> /Input Filter And Slow Start/AC_L_FUSED
- K1 pad 4: /Input Filter And Slow Start/AC_L_OUT -> /Input Filter And Slow Start/AC_L_INPUT_RELAY
- L1 pad 1: Net-(C6-Pad1) -> /POS_RECTIFIED
- L1 pad 2: /AC_N -> +70V
- Q1 pad 1: /L_SW_NODE -> /EN/NC
- Q1 pad 2: Net-(Q1-S) -> Net-(Q1-B)
- Q1 pad 3: /LS -> PRIM_SGND
- Q2 pad 1: VBUS -> Net-(D5-K)
- Q2 pad 2: /H_SW_NODE -> Net-(Q2-G)
- Q2 pad 3: /HS -> PRIM_SGND
- R1 pad 1: +12V -> /PRIM_MUX_SELECT
- R1 pad 2: Net-(K1-COIL_2) -> Net-(R1-Pad2)
- R10 pad 1: /VREF -> +3V3_Secondary
- R10 pad 2: PRIM_SGND -> /~{PRIM_OVP}
- R12 pad 1: +5V_Primary -> Net-(Q1-B)
- R12 pad 2: /GATE_DRIVER_HI -> PRIM_SGND
- R13 pad 1: +5V_Primary -> +12V_Primary
- R13 pad 2: /GATE_DRIVER_LI -> Net-(U4-VDD)
- R14 pad 1: VBUS -> Net-(U4-VDD)
- R14 pad 2: Net-(U5-EN/UV) -> Net-(D4-A)
- R15 pad 1: Net-(D11-Pad2) -> Net-(D4-A)
- R15 pad 2: Net-(D12-K) -> Net-(Q2-G)
- R17 pad 1: Net-(D15-A) -> Net-(Q2-G)
- R17 pad 2: Net-(R17-Pad2) -> PRIM_SGND
- R18 pad 1: Net-(R17-Pad2) -> Net-(Q3-G)
- R2 pad 1: /Input Filter And Slow Start/L_FILTERED -> /RELAY_SOFT_SWITCH
- R2 pad 2: /Input Filter And Slow Start/AC_L_OUT -> Net-(R2-Pad2)
- R24 pad 1: +3V3_Secondary -> Net-(U7-QA)
- R24 pad 2: /#GATE_DRIVER_ACTIVE -> Net-(D11-A)
- R29 pad 1: /Startup Power/BUCK_5V -> Net-(U7-QF)
- R29 pad 2: /Startup Power/FB -> Net-(D16-A)
- R3 pad 1: /Input Filter And Slow Start/COIL_GATE -> /RELAY_SWITCH
- R3 pad 2: /Input Filter And Slow Start/RELAY_SWITCH -> Net-(R3-Pad2)
- R30 pad 1: /Startup Power/FB -> Net-(U7-QG)
- R30 pad 2: SEC_SGND -> Net-(D17-A)
- R32 pad 1: +70V -> SEC_SHUNT_L
- R32 pad 2: Net-(C100-Pad2) -> SEC_SHUNT_H
- R33 pad 1: Net-(C100-Pad2) -> +70V
- R33 pad 2: -70V -> SEC_SHUNT_H
- R39 pad 1: Net-(U16-QA) -> +3V3_Secondary
- R39 pad 2: Net-(D18-A) -> Net-(C22-Pad1)
- R4 pad 1: /Input Filter And Slow Start/COIL_GATE -> PRIM_OCP
- R4 pad 2: PRIM_SGND -> Net-(R4-Pad2)
- R40 pad 1: Net-(U16-QB) -> +3V3_Secondary
- R40 pad 2: Net-(D19-A) -> Net-(C23-Pad1)
- R41 pad 1: Net-(U16-QC) -> SEC_SHUNT_H
- R41 pad 2: Net-(D20-A) -> /Current Sensing/+
- R42 pad 1: Net-(U16-QD) -> SEC_SHUNT_L
- R42 pad 2: Net-(D21-A) -> /Current Sensing/-
- R43 pad 1: Net-(U16-QE) -> PRIM_SHUNT_H
- R43 pad 2: Net-(D22-A) -> Net-(U10-+)
- R44 pad 1: Net-(U16-QF) -> PRIM_SHUNT_L
- R44 pad 2: Net-(D23-A) -> Net-(U10--)
- R45 pad 1: Net-(U16-QG) -> Net-(C22-Pad1)
- R45 pad 2: Net-(D24-A) -> /Current Sensing/AD_TEMP_DIODE1
- R46 pad 1: Net-(U16-QH) -> Net-(C23-Pad1)
- R46 pad 2: Net-(D25-A) -> /Current Sensing/AD_TEMP_NMOS_LS
- R6 pad 2: /VREF -> ~{PRIM_MUX_SELECT}
- SW1 pad 2: /MCU/~{RST} -> /MCU/~{MR}
- T1 pad 4: Net-(D12-A) -> Net-(D36-A)
- T1 pad 5: Net-(D13-A) -> /Startup Power/AUX_PRIM
- T1 pad 6: Net-(D14-A) -> /Startup Power/AUX_SEC
- U1 pad 1: /GATE_DRIVER_HI -> Net-(R1-Pad2)
- U1 pad 11: /HS -> PRIM_SGND
- U1 pad 12: /H_SW -> /~{RELAY_SWITCH}
- U1 pad 13: Net-(D16-K) -> PRIM_SGND
- U1 pad 14: unconnected-(U1-NC-Pad14) -> /~{RELAY_SOFT_SWITCH}
- U1 pad 2: /GATE_DRIVER_LI -> SEC_SGND
- U1 pad 3: PRIM_SGND -> Net-(R2-Pad2)
- U1 pad 4: /EN/NC -> SEC_SGND
- U1 pad 5: /LS -> Net-(R3-Pad2)
- U1 pad 6: /LO_SW -> SEC_SGND
- U1 pad 7: Net-(U1-VDD) -> unconnected-(U1-Pad7)
- U10 pad 1: /~{DISABLE_GATE_DRIVER} -> /Current Sensing/PRIMARY_CURRENT_SENSE
- U10 pad 2: SEC_SGND -> PRIM_SGND
- U10 pad 3: /~{ENABLE_GATE_DRIVER} -> Net-(U10-+)
- U10 pad 4: SEC_SGND -> Net-(U10--)
- U10 pad 5: (no net) -> +5V_Primary
- U11 pad 1: unconnected-(U11-Pad1) -> /Current Sensing/SECONDARY_CURRENT_SENSE
- U11 pad 2: unconnected-(U11-Pad2) -> SEC_SGND
- U11 pad 3: unconnected-(U11-Pad3) -> /Current Sensing/+
- U11 pad 4: unconnected-(U11-Pad4) -> /Current Sensing/-
- U11 pad 5: unconnected-(U11-Pad5) -> +3V3_Secondary
- U12 pad 1: unconnected-(U12-VBAT-Pad1) -> /Current Sensing/PRIM_CURRENT_SENSE
- U12 pad 2: unconnected-(U12-PC13-Pad2) -> PRIM_SGND
- U12 pad 3: unconnected-(U12-PC14-Pad3) -> /Current Sensing/PRIM_BUS_VOLTAGE
- U12 pad 4: unconnected-(U12-PC15-Pad4) -> /Current Sensing/PRIMARY_MUX_OUT
- U12 pad 5: unconnected-(U12-PD0-Pad5) -> +5V_Primary
- U12 pad 6: unconnected-(U12-PD1-Pad6) -> PRIM_MUX_SELECT
- U15 pad 1: /MCU/D- -> Net-(U15-+)
- U15 pad 3: /MCU/D+ -> Net-(U15--)
- U15 pad 4: /MCU/D+ -> /Current Sensing/MUX_OUT
- U15 pad 5: VBUS_USB -> +3V3_Secondary
- U3 pad 1: /Current Sensing/PRIMARY_CURRENT_SENSE -> Net-(R4-Pad2)
- U3 pad 3: /Current Sensing/+ -> Net-(R5-Pad2)
- U3 pad 4: /Current Sensing/- -> PRIM_SGND
- U3 pad 5: +5V -> SEC_SGND
- U4 pad 1: (no net) -> /GATE_DRIVER_HI_ISO
- U4 pad 10: (no net) -> unconnected-(U4-NC-Pad10)
- U4 pad 11: (no net) -> /HS
- U4 pad 12: (no net) -> /H_SW
- U4 pad 2: (no net) -> /GATE_DRIVER_LO_ISO
- U4 pad 3: (no net) -> PRIM_SGND
- U4 pad 4: (no net) -> /EN/NC
- U4 pad 5: /~{ENABLE_GATE_DRIVER} -> /LS
- U4 pad 6: SEC_SGND -> /L_SW
- U4 pad 7: PRIM_SGND -> Net-(U4-VDD)
- U4 pad 8: /EN/NC -> unconnected-(U4-NC-Pad8)
- U4 pad 9: (no net) -> unconnected-(U4-NC-Pad9)
- U5 pad 1: Net-(U5-EN/UV) -> /L_SW_NODE
- U5 pad 2: Net-(U5-BP/M) -> unconnected-(U5-Pad2)
- U5 pad 4: Net-(D12-A) -> unconnected-(U5-Pad4)
- U5 pad 5: GND1 -> unconnected-(U5-Pad5)
- U5 pad 6: GND1 -> unconnected-(U5-Pad6)
- U5 pad 7: GND1 -> unconnected-(U5-Pad7)
- U5 pad 8: GND1 -> unconnected-(U5-Pad8)
- U6 pad 1: Net-(R17-Pad2) -> /S11
- U6 pad 2: PRIM_SGND -> /S12
- U6 pad 3: GND1 -> /~{E}1
- U6 pad 4: Net-(U5-EN/UV) -> /S20
- U7 pad 1: +12V_Secondary -> Net-(U7-QB)
- U7 pad 2: PRIM_SGND -> Net-(U7-QC)
- U7 pad 3: +5V_Primary -> Net-(U7-QD)
- U8 pad 1: SEC_SGND -> /Current Sensing/AD_TEMP_NMOS_HS
- U8 pad 2: /Startup Power/SW -> /Current Sensing/AD_TEMP_TANSFORMER
- U8 pad 3: +12V_Secondary -> /TEMP_MUX1
- U8 pad 4: /Startup Power/FB -> /Current Sensing/AD_TEMP_DIODE_PRIM1
- U8 pad 5: +12V_Secondary -> /Current Sensing/AD_TEMP_NMOS_LS
- U8 pad 6: /Startup Power/BOOTSTRAP -> /~{E}1
- U9 pad 1: +5V_Secondary -> /Y4
- U9 pad 2: SEC_SGND -> /Y6
- U9 pad 3: +3V3_Secondary -> /TEMP_MUX2
Routing:
- net /Input Filter And Slow Start/AC_L_OUT: track 0.00 -> 94.3 mm
- net VBUS: track 0.00 -> 78.4 mm
- net /Input Filter And Slow Start/AC_L_INPUT_RELAY: track 0.00 -> 67.1 mm
- net /AC_N: track 0.00 -> 61.7 mm
- net /Input Filter And Slow Start/AC_L_FILTERED: track 0.00 -> 49.4 mm
- net /Input Filter And Slow Start/AC_N_OUT: track 0.00 -> 42.9 mm
- net /Input Filter And Slow Start/AC_L_FUSED: track 0.00 -> 19.0 mm
- net /AC_L: track 0.00 -> 13.5 mm
- net /Input Filter And Slow Start/AC_RELAY1_RC_SNUBBER_2: track 0.00 -> 5.41 mm
- net /Input Filter And Slow Start/AC_RELAY2_RC_SNUBBER_2: track 0.00 -> 4.39 mm
- net /Input Filter And Slow Start/AC_RELAY2_RC_SNUBBER_1: track 0.00 -> 3.72 mm
- net /Input Filter And Slow Start/AC_RELAY1_RC_SNUBBER_1: track 0.00 -> 3.72 mm
Other:
- board outline added: 187 x 352.1 mm
- copper layers 2 -> 4
