File: Rev_1/ECAD/power_board/sr_latch.kicad_sch (KiCad schematic)
At the start: 2 parts, among them U13 4001

Commit message: Assign footprints
Parts:
- C83: renamed from C41; footprint (none) -> Capacitor_SMD:C_0805_2012Metric
- renumbered U13 to U29
Changed lines of the file:
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@@
 		(dnp no)
 		(fields_autoplaced yes)
-		(property "Reference" "U13"
+		(property "Reference" "U29"
 			(at 144.78 34.29 90)
 			(show_name no)
@@
 			(project "power_board"
 				(path "/c8aad44b-d397-4b10-8f2c-430938609242/ff88370b-1696-4e04-941c-ae5f855f9f1d"
-					(reference "U13")
+					(reference "U29")
 					(unit 5)
 				)
@@
 		(dnp no)
 		(fields_autoplaced yes)
-		(property "Reference" "C41"
+		(property "Reference" "C83"
 			(at 144.78 21.59 90)
 			(show_name no)
@@
 			)
 		)
-		(property "Footprint" ""
+		(property "Footprint" "Capacitor_SMD:C_0805_2012Metric"
 			(at 148.59 28.2448 0)
 			(hide yes)
@@
 			(project "power_board"
 				(path "/c8aad44b-d397-4b10-8f2c-430938609242/ff88370b-1696-4e04-941c-ae5f855f9f1d"
-					(reference "C41")
+					(reference "C83")
 					(unit 1)
 				)
@@
 		(in_pos_files yes)
 		(dnp no)
-		(property "Reference" "#PWR029"
+		(property "Reference" "#PWR0191"
 			(at 130.556 24.384 0)
 			(hide yes)
@@
 			(project "power_board"
 				(path "/c8aad44b-d397-4b10-8f2c-430938609242/ff88370b-1696-4e04-941c-ae5f855f9f1d"
-					(reference "#PWR029")
+					(reference "#PWR0191")
 					(unit 1)
 				)
@@
 		(dnp no)
 		(fields_autoplaced yes)
-		(property "Reference" "U13"
+		(property "Reference" "U29"
 			(at 88.9 63.5 0)
 			(show_name no)
@@
 			(project "power_board"
 				(path "/c8aad44b-d397-4b10-8f2c-430938609242/ff88370b-1696-4e04-941c-ae5f855f9f1d"
-					(reference "U13")
+					(reference "U29")
 					(unit 2)
 				)
@@
 		(dnp no)
 		(fields_autoplaced yes)
-		(property "Reference" "U13"
+		(property "Reference" "U29"
 			(at 88.9 45.72 0)
 			(show_name no)
@@
 			(project "power_board"
 				(path "/c8aad44b-d397-4b10-8f2c-430938609242/ff88370b-1696-4e04-941c-ae5f855f9f1d"
-					(reference "U13")
+					(reference "U29")
 					(unit 1)
 				)
@@
 		(in_pos_files yes)
 		(dnp no)
-		(property "Reference" "#PWR030"
+		(property "Reference" "#PWR0192"
 			(at 158.496 44.196 0)
 			(hide yes)
@@
 			(project "power_board"
 				(path "/c8aad44b-d397-4b10-8f2c-430938609242/ff88370b-1696-4e04-941c-ae5f855f9f1d"
-					(reference "#PWR030")
+					(reference "#PWR0192")
 					(unit 1)
 				)

Commit message: Before PR
Parts:
- removed C83: 100n, Capacitor_SMD:C_0805_2012Metric, symbol Device:C
- removed U29: 4001, symbol 4xxx:4001
Other:
- note removed: "GROUNDING?"
