File: Rev_1/ECAD/power_board/startup_power.kicad_sch (KiCad schematic)
At the start: 33 parts, among them T1 063932, U5 TNY274P, U6 PC817, U7 5V LDO, U8 LMR51430, U9 3v3 LDO

Commit message: Assign footprints
Parts:
- added C58: 10u, 50V, symbol Device:C_Small
- added C67, C69, C70: 1u, symbol Device:C_Small
- added U24: TPS60403DBV, Package_TO_SOT_SMD:SOT-23-5, symbol Regulator_SwitchedCapacitor:TPS60403DBV
- renumbered C4 to C56, C5 to C57, C12 to C59, C13 to C60, C14 to C61, C21 to C62, C22 to C63, C23 to C64, C24 to C65, C25 to C66, C26 to C68, C27 to C71, D11 to D31, D12 to D32, D13 to D33, D14 to D34, D15 to D35, D7 to D36, D8 to D37, R14 to R92, R15 to R93, R16 to R94, R17 to R95, R18 to R96, R29 to R97, R30 to R98, U5 to U20, U6 to U21, U7 to U22, U8 to U23, U9 to U25
Connections:
- net +5V_Secondary: now also C67.1, U24.2 (IN)
- net GND1: now also C58.2
- net SEC_SGND: now also C67.2, C70.2, U24.4 (GND)
- net at C57.1, U20.2 (BP/M): now also C58.1
- new net: C69.1, U24.5 (C_{FLY+})
- new net: C69.2, U24.3 (C_{FLY-})
- new net -5V: C70.1, U24.1 (OUT)
Other:
- note added: "-5V - Secondary"

Commit message: Before PR
Parts:
- removed C58: 10u, 50V, symbol Device:C_Small
- added C53: 10u, 50V, Capacitor_THT:CP_Radial_D5.0mm_P2.00mm, symbol Device:C_Polarized_Small
- added C57: 2n2, Capacitor_THT:C_Rect_L18.0mm_W6.0mm_P15.00mm_FKS3_FKP3, symbol Device:C_Small
- added NT3, NT4: NetTie_2, symbol Device:NetTie_2
- C51: renamed from C56; footprint (none) -> Capacitor_SMD:C_1206_3216Metric; Mouser No: (none) -> 791-1206B103M102CT
- C52: renamed from C57; footprint (none) -> Capacitor_SMD:C_0805_2012Metric; Mouser No: (none) -> 603-CC603KRX5R9BB104; Part-DB ID (none) -> 25; Part-DB NAME (none) -> C0805C104M5RACTU
- C55: renamed from C60; value 1000u -> 470u; footprint (none) -> Capacitor_THT:C_Radial_D10.0mm_H16.0mm_P5.00mm
- C56: renamed from C61; value 1000u -> 470u; footprint (none) -> Capacitor_THT:C_Radial_D10.0mm_H16.0mm_P5.00mm
- C58: renamed from C62; footprint (none) -> Capacitor_SMD:C_0805_2012Metric; Mouser No: (none) -> 791-0805X475M250CT
- C59: renamed from C63; value 10u -> 10u, 6V3; Part-DB ID (none) -> 6; Part-DB NAME (none) -> CL21A106KQFNNWE
- C60: renamed from C64; Part-DB ID (none) -> 5; Part-DB NAME (none) -> CL21A226MAYNNNE
- C62: renamed from C66; footprint (none) -> Capacitor_SMD:C_1206_3216Metric
- C63: renamed from C67; value 1u -> 1u, 16VDC; footprint (none) -> Capacitor_SMD:C_0805_2012Metric; Part-DB ID (none) -> 36; Part-DB NAME (none) -> 0805B105K160CT
- C64: renamed from C68; value 10u -> 10u, 6V3; Part-DB ID (none) -> 6; Part-DB NAME (none) -> CL21A106KQFNNWE
- C65: renamed from C69; value 1u -> 1u, 16VDC; footprint (none) -> Capacitor_SMD:C_0805_2012Metric; Part-DB ID (none) -> 36; Part-DB NAME (none) -> 0805B105K160CT
- C66: renamed from C70; value 1u -> 1u, 16VDC; footprint (none) -> Capacitor_SMD:C_0805_2012Metric; Part-DB ID (none) -> 36; Part-DB NAME (none) -> 0805B105K160CT
- C67: renamed from C71; Part-DB ID (none) -> 5; Part-DB NAME (none) -> CL21A226MAYNNNE
- D35: renamed from D31; footprint (none) -> Diode_THT:D_DO-15_P10.16mm_Horizontal; Mouser No: (none) -> 576-P6KE150A
- D37: renamed from D33; value D_Schottky -> SB24; footprint Diode_SMD:D_1206_3216Metric -> Diode_SMD:D_SOD-128; Mouser No: (none) -> 241-SB24AFCAUR1000A1
- D38: renamed from D34; value D_Schottky -> SB24; footprint Diode_SMD:D_1206_3216Metric -> Diode_SMD:D_SOD-128; Mouser No: (none) -> 241-SB24AFCAUR1000A1
- D39: renamed from D35; footprint (none) -> Diode_THT:D_DO-35_SOD27_P7.62mm_Horizontal; Mouser No: (none) -> 512-BZX79C11
- D40: renamed from D36; value D_Schottky -> SK15; footprint (none) -> Diode_SMD:D_SMA_Handsoldering
- D41: renamed from D37; value D_Schottky -> SK15; footprint (none) -> Diode_SMD:D_SMA_Handsoldering
- R100: renamed from R92; value 3.6M -> 3.6M, 325V; footprint Resistor_SMD:R_0805_2012Metric -> Resistor_THT:R_Axial_DIN0309_L9.0mm_D3.2mm_P12.70mm_Horizontal; Mouser No: (none) -> 603-CFR-50JB-52-3M6
- R101: renamed from R93; Part-DB ID (none) -> 66; Part-DB NAME (none) -> 40819310
- R102: renamed from R94; value 100 -> 100, 325V; footprint (none) -> Resistor_THT:R_Axial_DIN0411_L9.9mm_D3.6mm_P12.70mm_Horizontal; Mouser No: (none) -> 708-RSMF1JT100R
- R105: renamed from R97; footprint Resistor_SMD:R_0805_2012Metric -> Resistor_SMD:R_0603_1608Metric
- U17: renamed from U21; footprint Package_DIP:DIP-4_W7.62mm -> Package_SO:SOP-4_4.4x2.6mm_P1.27mm; Mouser No: (none) -> 852-PC817X1CSP9F
- U20: renamed from U24; Part-DB ID (none) -> 48; Part-DB NAME (none) -> TPS60403DBVRG4
- renumbered C59 to C54, C65 to C61, D32 to D36, R95 to R103, R96 to R104, R98 to R106, U20 to U16, U22 to U18, U23 to U19, U25 to U21
Connections:
- net +12V_Primary: now also C59.1, U18.1 (IN)
- net +12V_Secondary: no longer C59.1, U18.1 (IN)
- net GND1: now also C53.2, C57.1, NT3.2
- net PRIM_SGND: now also C57.2, NT3.1
- net SEC_SGND: now also NT4.1
- net at C52.1, U16.2 (BP/M): now also C53.1
- net AUX_PRIM: now reaches D37.2 (A), T1.5
- net AUX_SEC: now reaches D38.2 (A), T1.6
- new net GND2: NT4.2
